File: kicad/IR_RCV.sch (KiCad schematic (older format))
At the start: 10 parts, among them J15 Host, J16 Slave, Q1 MTM231232LBF, Q2 DMN3065LW-7, Q3 SFH3015FA

Commit message: 部品を配置
Parts:
- renumbered J15 to J14, J16 to J15
Changed lines of the file:
@@
 EESchema Schematic File Version 4
 LIBS:KERISE-cache
-EELAYER 26 0
+EELAYER 29 0
 EELAYER END
 $Descr A4 11693 8268
 encoding utf-8
-Sheet 12 15
+Sheet 5 13
 Title ""
 Date ""
@@
 AR Path="/57CF0B09/589BE75A" Ref="Q2"  Part="1"
 AR Path="/57CF2A30/589BE75A" Ref="Q5"  Part="1"
-AR Path="/597E1B35/589BE75A" Ref="Q9"  Part="1"
-AR Path="/597E1B39/589BE75A" Ref="Q12"  Part="1"
-F 0 "Q12" H 4300 5650 50  0000 R CNN
+AR Path="/597E1B35/589BE75A" Ref="Q8"  Part="1"
+AR Path="/597E1B39/589BE75A" Ref="Q11"  Part="1"
+F 0 "Q11" H 4300 5650 50  0000 R CNN
 F 1 "DMN3065LW-7" H 4350 5350 50  0000 R CNN
 F 2 "mouse:SOT-323_SC-70" H 4500 5600 50  0001 C CNN
@@
 AR Path="/57CF0B09/589BE76D" Ref="R6"  Part="1"
 AR Path="/57CF2A30/589BE76D" Ref="R8"  Part="1"
-AR Path="/597E1B35/589BE76D" Ref="R11"  Part="1"
-AR Path="/597E1B39/589BE76D" Ref="R13"  Part="1"
-F 0 "R13" V 4480 4450 50  0000 C CNN
+AR Path="/597E1B35/589BE76D" Ref="R10"  Part="1"
+AR Path="/597E1B39/589BE76D" Ref="R12"  Part="1"
+F 0 "R12" V 4480 4450 50  0000 C CNN
 F 1 "100" V 4400 4450 50  0000 C CNN
 F 2 "Resistor_SMD:R_0603_1608Metric" V 4330 4450 50  0001 C CNN
@@
 AR Path="/57CF0B09/589BF265" Ref="#PWR041"  Part="1"
 AR Path="/57CF2A30/589BF265" Ref="#PWR044"  Part="1"
-AR Path="/597E1B35/589BF265" Ref="#PWR062"  Part="1"
-AR Path="/597E1B39/589BF265" Ref="#PWR065"  Part="1"
-F 0 "#PWR065" H 4400 2350 50  0001 C CNN
+AR Path="/597E1B35/589BF265" Ref="#PWR052"  Part="1"
+AR Path="/597E1B39/589BF265" Ref="#PWR055"  Part="1"
+F 0 "#PWR055" H 4400 2350 50  0001 C CNN
 F 1 "GND" H 4400 2450 50  0000 C CNN
 F 2 "" H 4400 2600 50  0000 C CNN
@@
 AR Path="/57CF0B09/59C54857" Ref="#PWR039"  Part="1"
 AR Path="/57CF2A30/59C54857" Ref="#PWR042"  Part="1"
-AR Path="/597E1B35/59C54857" Ref="#PWR060"  Part="1"
-AR Path="/597E1B39/59C54857" Ref="#PWR063"  Part="1"
-F 0 "#PWR063" H 4100 1850 50  0001 C CNN
+AR Path="/597E1B35/59C54857" Ref="#PWR050"  Part="1"
+AR Path="/597E1B39/59C54857" Ref="#PWR053"  Part="1"
+F 0 "#PWR053" H 4100 1850 50  0001 C CNN
 F 1 "VDDA" H 4100 2150 50  0000 C CNN
 F 2 "" H 4100 2000 50  0001 C CNN
@@
 AR Path="/57CF0B09/5A172FEF" Ref="#PWR040"  Part="1"
 AR Path="/57CF2A30/5A172FEF" Ref="#PWR043"  Part="1"
-AR Path="/597E1B35/5A172FEF" Ref="#PWR061"  Part="1"
-AR Path="/597E1B39/5A172FEF" Ref="#PWR064"  Part="1"
-F 0 "#PWR064" H 4400 1850 50  0001 C CNN
+AR Path="/597E1B35/5A172FEF" Ref="#PWR051"  Part="1"
+AR Path="/597E1B39/5A172FEF" Ref="#PWR054"  Part="1"
+F 0 "#PWR054" H 4400 1850 50  0001 C CNN
 F 1 "+3.3V" H 4400 2140 50  0000 C CNN
 F 2 "" H 4400 2000 50  0001 C CNN
@@
 AR Path="/57CF0B09/5A1B992B" Ref="C9"  Part="1"
 AR Path="/57CF2A30/5A1B992B" Ref="C11"  Part="1"
-AR Path="/597E1B35/5A1B992B" Ref="C18"  Part="1"
-AR Path="/597E1B39/5A1B992B" Ref="C20"  Part="1"
-F 0 "C20" H 5025 5650 50  0000 L CNN
+AR Path="/597E1B35/5A1B992B" Ref="C15"  Part="1"
+AR Path="/597E1B39/5A1B992B" Ref="C17"  Part="1"
+F 0 "C17" H 5025 5650 50  0000 L CNN
 F 1 "1u" H 5025 5450 50  0000 L CNN
 F 2 "Capacitor_SMD:C_0402_1005Metric" H 5038 5400 50  0001 C CNN
@@
 AR Path="/57CF0B09/5A4ADF8B" Ref="Q3"  Part="1"
 AR Path="/57CF2A30/5A4ADF8B" Ref="Q6"  Part="1"
-AR Path="/597E1B35/5A4ADF8B" Ref="Q10"  Part="1"
-AR Path="/597E1B39/5A4ADF8B" Ref="Q13"  Part="1"
-F 0 "Q13" H 5700 4450 50  0000 L CNN
+AR Path="/597E1B35/5A4ADF8B" Ref="Q9"  Part="1"
+AR Path="/597E1B39/5A4ADF8B" Ref="Q12"  Part="1"
+F 0 "Q12" H 5700 4450 50  0000 L CNN
 F 1 "SFH3015FA" H 5700 4350 50  0000 L CNN
 F 2 "mouse:SFH3015FA" H 5700 4500 50  0001 C CNN
@@
 AR Path="/57CF0B09/589BEE3B" Ref="R7"  Part="1"
 AR Path="/57CF2A30/589BEE3B" Ref="R9"  Part="1"
-AR Path="/597E1B35/589BEE3B" Ref="R12"  Part="1"
-AR Path="/597E1B39/589BEE3B" Ref="R14"  Part="1"
-F 0 "R14" V 5680 5550 50  0000 C CNN
+AR Path="/597E1B35/589BEE3B" Ref="R11"  Part="1"
+AR Path="/597E1B39/589BEE3B" Ref="R13"  Part="1"
+F 0 "R13" V 5680 5550 50  0000 C CNN
 F 1 "10k" V 5600 5550 50  0000 C CNN
 F 2 "Resistor_SMD:R_0201_0603Metric" V 5530 5550 50  0001 C CNN
@@
 AR Path="/57CF0B09/5AB4DD07" Ref="Q1"  Part="1"
 AR Path="/57CF2A30/5AB4DD07" Ref="Q4"  Part="1"
-AR Path="/597E1B35/5AB4DD07" Ref="Q8"  Part="1"
-AR Path="/597E1B39/5AB4DD07" Ref="Q11"  Part="1"
-F 0 "Q11" H 4500 4050 50  0000 L CNN
+AR Path="/597E1B35/5AB4DD07" Ref="Q7"  Part="1"
+AR Path="/597E1B39/5AB4DD07" Ref="Q10"  Part="1"
+F 0 "Q10" H 4500 4050 50  0000 L CNN
 F 1 "MTM231232LBF" H 4500 3950 50  0000 L CNN
 F 2 "mouse:SOT-323_SC-70" H 4500 4100 50  0001 C CNN
@@
 	4000 5500 4100 5500
 $Comp
-L Connector:Conn_01x05_Female J15
+L Connector:Conn_01x05_Female J14
 U 1 1 5B6F3B71
 P 4700 2300
-AR Path="/597E1B39/5B6F3B71" Ref="J15"  Part="1"
-AR Path="/597E1B35/5B6F3B71" Ref="J13"  Part="1"
+AR Path="/597E1B39/5B6F3B71" Ref="J14"  Part="1"
+AR Path="/597E1B35/5B6F3B71" Ref="J12"  Part="1"
 AR Path="/57CF0B09/5B6F3B71" Ref="J3"  Part="1"
 AR Path="/57CF2A30/5B6F3B71" Ref="J5"  Part="1"
-F 0 "J15" H 4728 2326 50  0000 L CNN
+F 0 "J14" H 4728 2326 50  0000 L CNN
 F 1 "Host" H 4728 2235 50  0000 L CNN
 F 2 "mouse:STAND_HOST_05" H 4700 2300 50  0001 C CNN
@@
 $EndComp
 $Comp
-L Connector:Conn_01x05_Male J16
+L Connector:Conn_01x05_Male J15
 U 1 1 5B6F3C20
 P 5000 2300
-AR Path="/597E1B39/5B6F3C20" Ref="J16"  Part="1"
-AR Path="/597E1B35/5B6F3C20" Ref="J14"  Part="1"
+AR Path="/597E1B39/5B6F3C20" Ref="J15"  Part="1"
+AR Path="/597E1B35/5B6F3C20" Ref="J13"  Part="1"
 AR Path="/57CF0B09/5B6F3C20" Ref="J4"  Part="1"
 AR Path="/57CF2A30/5B6F3C20" Ref="J6"  Part="1"
-F 0 "J16" H 5106 2678 50  0000 C CNN
+F 0 "J15" H 5106 2678 50  0000 C CNN
 F 1 "Slave" H 5106 2587 50  0000 C CNN
 F 2 "mouse:STAND_SLAVE_05" H 5000 2300 50  0001 C CNN
@@
 AR Path="/57CF2A30/5C29B79F" Ref="C12"  Part="1"
 AR Path="/57CF0B09/5C29B79F" Ref="C10"  Part="1"
-AR Path="/597E1B35/5C29B79F" Ref="C19"  Part="1"
-AR Path="/597E1B39/5C29B79F" Ref="C21"  Part="1"
-F 0 "C21" H 6692 4846 50  0000 L CNN
+AR Path="/597E1B35/5C29B79F" Ref="C16"  Part="1"
+AR Path="/597E1B39/5C29B79F" Ref="C18"  Part="1"
+F 0 "C18" H 6692 4846 50  0000 L CNN
 F 1 "0.1u" H 6692 4755 50  0000 L CNN
 F 2 "Capacitor_SMD:C_0201_0603Metric" H 6600 4800 50  0001 C CNN

Commit message: 配線幅を改良
Changed lines of the file:
@@
 $Descr A4 11693 8268
 encoding utf-8
-Sheet 5 13
+Sheet 4 13
 Title ""
 Date ""
@@
 AR Path="/597E1B35/589BE75A" Ref="Q8"  Part="1"
 AR Path="/597E1B39/589BE75A" Ref="Q11"  Part="1"
-F 0 "Q11" H 4300 5650 50  0000 R CNN
+F 0 "Q2" H 4300 5650 50  0000 R CNN
 F 1 "DMN3065LW-7" H 4350 5350 50  0000 R CNN
 F 2 "mouse:SOT-323_SC-70" H 4500 5600 50  0001 C CNN
@@
 AR Path="/597E1B35/589BE76D" Ref="R10"  Part="1"
 AR Path="/597E1B39/589BE76D" Ref="R12"  Part="1"
-F 0 "R12" V 4480 4450 50  0000 C CNN
+F 0 "R6" V 4480 4450 50  0000 C CNN
 F 1 "100" V 4400 4450 50  0000 C CNN
 F 2 "Resistor_SMD:R_0603_1608Metric" V 4330 4450 50  0001 C CNN
@@
 AR Path="/597E1B35/589BF265" Ref="#PWR052"  Part="1"
 AR Path="/597E1B39/589BF265" Ref="#PWR055"  Part="1"
-F 0 "#PWR055" H 4400 2350 50  0001 C CNN
+F 0 "#PWR041" H 4400 2350 50  0001 C CNN
 F 1 "GND" H 4400 2450 50  0000 C CNN
 F 2 "" H 4400 2600 50  0000 C CNN
@@
 AR Path="/597E1B35/594AC674" Ref="D5"  Part="1"
 AR Path="/597E1B39/594AC674" Ref="D6"  Part="1"
-F 0 "D6" V 4500 4800 50  0000 C CNN
+F 0 "D3" V 4500 4800 50  0000 C CNN
 F 1 "SFH4045N" V 4400 4650 50  0000 C CNN
 F 2 "mouse:SFH4045N" H 4400 4950 50  0001 C CNN
@@
 AR Path="/597E1B35/59C54857" Ref="#PWR050"  Part="1"
 AR Path="/597E1B39/59C54857" Ref="#PWR053"  Part="1"
-F 0 "#PWR053" H 4100 1850 50  0001 C CNN
+F 0 "#PWR039" H 4100 1850 50  0001 C CNN
 F 1 "VDDA" H 4100 2150 50  0000 C CNN
 F 2 "" H 4100 2000 50  0001 C CNN
@@
 AR Path="/597E1B35/5A172FEF" Ref="#PWR051"  Part="1"
 AR Path="/597E1B39/5A172FEF" Ref="#PWR054"  Part="1"
-F 0 "#PWR054" H 4400 1850 50  0001 C CNN
+F 0 "#PWR040" H 4400 1850 50  0001 C CNN
 F 1 "+3.3V" H 4400 2140 50  0000 C CNN
 F 2 "" H 4400 2000 50  0001 C CNN
@@
 AR Path="/597E1B35/5A1B992B" Ref="C15"  Part="1"
 AR Path="/597E1B39/5A1B992B" Ref="C17"  Part="1"
-F 0 "C17" H 5025 5650 50  0000 L CNN
+F 0 "C9" H 5025 5650 50  0000 L CNN
 F 1 "1u" H 5025 5450 50  0000 L CNN
 F 2 "Capacitor_SMD:C_0402_1005Metric" H 5038 5400 50  0001 C CNN
@@
 AR Path="/597E1B35/5A4ADF8B" Ref="Q9"  Part="1"
 AR Path="/597E1B39/5A4ADF8B" Ref="Q12"  Part="1"
-F 0 "Q12" H 5700 4450 50  0000 L CNN
+F 0 "Q3" H 5700 4450 50  0000 L CNN
 F 1 "SFH3015FA" H 5700 4350 50  0000 L CNN
 F 2 "mouse:SFH3015FA" H 5700 4500 50  0001 C CNN
@@
 AR Path="/597E1B35/589BEE3B" Ref="R11"  Part="1"
 AR Path="/597E1B39/589BEE3B" Ref="R13"  Part="1"
-F 0 "R13" V 5680 5550 50  0000 C CNN
+F 0 "R7" V 5680 5550 50  0000 C CNN
 F 1 "10k" V 5600 5550 50  0000 C CNN
 F 2 "Resistor_SMD:R_0201_0603Metric" V 5530 5550 50  0001 C CNN
@@
 AR Path="/597E1B35/5AB4DD07" Ref="Q7"  Part="1"
 AR Path="/597E1B39/5AB4DD07" Ref="Q10"  Part="1"
-F 0 "Q10" H 4500 4050 50  0000 L CNN
+F 0 "Q1" H 4500 4050 50  0000 L CNN
 F 1 "MTM231232LBF" H 4500 3950 50  0000 L CNN
 F 2 "mouse:SOT-323_SC-70" H 4500 4100 50  0001 C CNN
@@
 AR Path="/57CF0B09/5B6F3B71" Ref="J3"  Part="1"
 AR Path="/57CF2A30/5B6F3B71" Ref="J5"  Part="1"
-F 0 "J14" H 4728 2326 50  0000 L CNN
+F 0 "J3" H 4728 2326 50  0000 L CNN
 F 1 "Host" H 4728 2235 50  0000 L CNN
 F 2 "mouse:STAND_HOST_05" H 4700 2300 50  0001 C CNN
@@
 AR Path="/57CF0B09/5B6F3C20" Ref="J4"  Part="1"
 AR Path="/57CF2A30/5B6F3C20" Ref="J6"  Part="1"
-F 0 "J15" H 5106 2678 50  0000 C CNN
+F 0 "J4" H 5106 2678 50  0000 C CNN
 F 1 "Slave" H 5106 2587 50  0000 C CNN
 F 2 "mouse:STAND_SLAVE_05" H 5000 2300 50  0001 C CNN
@@
 AR Path="/597E1B35/5C29B79F" Ref="C16"  Part="1"
 AR Path="/597E1B39/5C29B79F" Ref="C18"  Part="1"
-F 0 "C18" H 6692 4846 50  0000 L CNN
+F 0 "C10" H 6692 4846 50  0000 L CNN
 F 1 "0.1u" H 6692 4755 50  0000 L CNN
 F 2 "Capacitor_SMD:C_0201_0603Metric" H 6600 4800 50  0001 C CNN
