File: kicad/IR_RCV.sch (KiCad schematic (older format))
At the start: 10 parts, among them J3 Host, J4 Slave, Q1 MTM231232LBF, Q2 DMN3065LW-7, Q3 SFH3015FA

Commit message: 予備配線完了
Parts:
- removed Q1: MTM231232LBF, mouse:SOT-323_SC-70, symbol Device:Q_PMOS_GSD
- D8: renamed from D3; footprint mouse:SFH4045N -> mouse:SFH4045N_L
- J12: renamed from J3; footprint mouse:IR_HOST_04 -> mouse:IR_HOST_V_04
- J13: renamed from J4; footprint mouse:IR_SLAVE_04 -> mouse:IR_SLAVE_V_04
- Q9: renamed from Q3; footprint mouse:SFH3015FA -> mouse:SFH3015FA_L
- renumbered C11 to C15, C8 to C16, Q2 to Q8, R6 to R11, R7 to R12
Connections:
- net s_3.3V: now also R11.1
Other:
- note added: "Photo Reflector v2020.02.20\nKERI's Lab"
- note removed: "Photo Reflector v2020.02.17\nKERI's Lab"
- moved on the sheet: C8, D5, Q2, Q3, R5, R6

Commit message: update kicad .gitignore
Parts:
- C16: value 2.2u -> 1u
Other:
- note added: "Photo Reflector"
- note removed: "Photo Reflector v2020.02.20\nKERI's Lab"
Changed lines of the file:
@@
 $Descr A4 11693 8268
 encoding utf-8
-Sheet 5 13
+Sheet 10 13
 Title ""
 Date ""
@@
 Text HLabel 4400 2800 0    60   Input ~ 0
 IR_RCV
-Text Notes 3500 3600 0    79   ~ 0
-Photo Reflector v2020.02.20\nKERI's Lab
 $Comp
 L Device:Q_NMOS_GSD Q8
@@
 AR Path="/597E1B35/589BE75A" Ref="Q4"  Part="1"
 AR Path="/597E1B39/589BE75A" Ref="Q2"  Part="1"
-F 0 "Q2" H 4300 5150 50  0000 R CNN
+F 0 "Q6" H 4300 5150 50  0000 R CNN
 F 1 "DMN3065LW-7" H 4350 4850 50  0000 R CNN
 F 2 "mouse:SOT-323_SC-70" H 4500 5100 50  0001 C CNN
@@
 AR Path="/597E1B35/589BE76D" Ref="R7"  Part="1"
 AR Path="/597E1B39/589BE76D" Ref="R5"  Part="1"
-F 0 "R5" V 4480 3950 50  0000 C CNN
+F 0 "R9" V 4480 3950 50  0000 C CNN
 F 1 "100" V 4400 3950 50  0000 C CNN
 F 2 "Resistor_SMD:R_0603_1608Metric" V 4330 3950 50  0001 C CNN
@@
 AR Path="/597E1B35/589BF265" Ref="#PWR028"  Part="1"
 AR Path="/597E1B39/589BF265" Ref="#PWR026"  Part="1"
-F 0 "#PWR037" H 4400 2750 50  0001 C CNN
+F 0 "#PWR035" H 4400 2750 50  0001 C CNN
 F 1 "GND" H 4400 2850 50  0000 C CNN
 F 2 "" H 4400 3000 50  0000 C CNN
@@
 AR Path="/597E1B35/594AC674" Ref="D6"  Part="1"
 AR Path="/597E1B39/594AC674" Ref="D5"  Part="1"
-F 0 "D5" V 4500 4300 50  0000 C CNN
+F 0 "D7" V 4500 4300 50  0000 C CNN
 F 1 "SFH4045N" V 4400 4150 50  0000 C CNN
 F 2 "mouse:SFH4045N_L" H 4400 4450 50  0001 C CNN
@@
 AR Path="/597E1B35/5A172FEF" Ref="#PWR027"  Part="1"
 AR Path="/597E1B39/5A172FEF" Ref="#PWR025"  Part="1"
-F 0 "#PWR036" H 4400 2350 50  0001 C CNN
+F 0 "#PWR034" H 4400 2350 50  0001 C CNN
 F 1 "+3.3V" H 4400 2640 50  0000 C CNN
 F 2 "" H 4400 2500 50  0001 C CNN
@@
 AR Path="/597E1B35/5A1B992B" Ref="C10"  Part="1"
 AR Path="/597E1B39/5A1B992B" Ref="C8"  Part="1"
-F 0 "C8" H 5025 5150 50  0000 L CNN
-F 1 "2.2u" H 5025 4950 50  0000 L CNN
+F 0 "C14" H 5025 5150 50  0000 L CNN
+F 1 "1u" H 5025 4950 50  0000 L CNN
 F 2 "Capacitor_SMD:C_0402_1005Metric" H 5038 4900 50  0001 C CNN
 F 3 "" H 5000 5050 50  0001 C CNN
@@
 AR Path="/597E1B35/5A4ADF8B" Ref="Q5"  Part="1"
 AR Path="/597E1B39/5A4ADF8B" Ref="Q3"  Part="1"
-F 0 "Q3" H 5700 4550 50  0000 L CNN
+F 0 "Q7" H 5700 4550 50  0000 L CNN
 F 1 "SFH3015FA" H 5700 4450 50  0000 L CNN
 F 2 "mouse:SFH3015FA_L" H 5700 4600 50  0001 C CNN
@@
 AR Path="/597E1B35/589BEE3B" Ref="R8"  Part="1"
 AR Path="/597E1B39/589BEE3B" Ref="R6"  Part="1"
-F 0 "R6" V 5680 5050 50  0000 C CNN
+F 0 "R10" V 5680 5050 50  0000 C CNN
 F 1 "10k" V 5600 5050 50  0000 C CNN
 F 2 "Resistor_SMD:R_0201_0603Metric" V 5530 5050 50  0001 C CNN
@@
 Wire Wire Line
 	5700 4800 5600 4800
-Wire Notes Line
-	3400 6100 6200 6100
 Wire Wire Line
 	4400 4800 4400 4600
 Wire Wire Line
 	5000 4200 5000 4900
-Wire Notes Line
-	3400 3300 3400 6100
-Wire Notes Line
-	3400 3300 6200 3300
-Wire Notes Line
-	6200 3300 6200 6100
 Wire Wire Line
 	4400 4200 4400 4100
@@
 AR Path="/597E1B35/5C29B79F" Ref="C11"  Part="1"
 AR Path="/597E1B39/5C29B79F" Ref="C9"  Part="1"
-F 0 "C9" H 6692 4846 50  0000 L CNN
+F 0 "C15" H 6692 4846 50  0000 L CNN
 F 1 "0.1u" H 6692 4755 50  0000 L CNN
 F 2 "Capacitor_SMD:C_0201_0603Metric" H 6600 4800 50  0001 C CNN
@@
 AR Path="/597E1B35/5E4BA6B8" Ref="J3"  Part="1"
 AR Path="/597E1B39/5E4BA6B8" Ref="J1"  Part="1"
-F 0 "J1" H 4728 2676 50  0000 L CNN
+F 0 "J10" H 4728 2676 50  0000 L CNN
 F 1 "Host" H 4728 2585 50  0000 L CNN
 F 2 "mouse:IR_HOST_V_04" H 4700 2700 50  0001 C CNN
@@
 AR Path="/597E1B35/5E4BAD76" Ref="J4"  Part="1"
 AR Path="/597E1B39/5E4BAD76" Ref="J2"  Part="1"
-F 0 "J2" H 5108 2981 50  0000 C CNN
+F 0 "J11" H 5108 2981 50  0000 C CNN
 F 1 "Slave" H 5108 2890 50  0000 C CNN
 F 2 "mouse:IR_SLAVE_V_04" H 5000 2700 50  0001 C CNN
@@
 Wire Wire Line
 	6600 5500 6600 4900
+Text Notes 3500 3600 0    79   ~ 0
+Photo Reflector
 $EndSCHEMATC

Commit message: KiCad: update pcb
Parts:
- C15: symbol Device:C_Small -> KERISE-rescue:C_Small-Device-KERISE-rescue-KERISE-rescue
- C16: symbol Device:C -> KERISE-rescue:C-Device-KERISE-rescue-KERISE-rescue
- D8: symbol Device:LED -> KERISE-rescue:LED-Device-KERISE-rescue-KERISE-rescue
- J12: symbol Connector:Conn_01x04_Female -> KERISE-rescue:Conn_01x04_Female-Connector-KERISE-rescue-KERISE-rescue
- J13: symbol Connector:Conn_01x04_Male -> KERISE-rescue:Conn_01x04_Male-Connector-KERISE-rescue-KERISE-rescue
- Q8: symbol Device:Q_NMOS_GSD -> KERISE-rescue:Q_NMOS_GSD-Device-KERISE-rescue-KERISE-rescue
- Q9: symbol Device:Q_Photo_NPN -> KERISE-rescue:Q_Photo_NPN-Device-KERISE-rescue-KERISE-rescue
- R11, R12: symbol Device:R -> KERISE-rescue:R-Device-KERISE-rescue-KERISE-rescue
Changed lines of the file:
@@
 $Descr A4 11693 8268
 encoding utf-8
-Sheet 10 13
+Sheet 6 13
 Title ""
 Date ""
@@
 IR_RCV
 $Comp
-L Device:Q_NMOS_GSD Q8
+L KERISE-rescue:Q_NMOS_GSD-Device-KERISE-rescue-KERISE-rescue Q8
 U 1 1 589BE75A
 P 4300 5000
@@
 AR Path="/597E1B35/589BE75A" Ref="Q4"  Part="1"
 AR Path="/597E1B39/589BE75A" Ref="Q2"  Part="1"
-F 0 "Q6" H 4300 5150 50  0000 R CNN
+AR Path="/589BE75A" Ref="Q?"  Part="1"
+F 0 "Q8" H 4300 5150 50  0000 R CNN
 F 1 "DMN3065LW-7" H 4350 4850 50  0000 R CNN
 F 2 "mouse:SOT-323_SC-70" H 4500 5100 50  0001 C CNN
@@
 $EndComp
 $Comp
-L Device:R R11
+L KERISE-rescue:R-Device-KERISE-rescue-KERISE-rescue R11
 U 1 1 589BE76D
 P 4400 3950
@@
 AR Path="/597E1B35/589BE76D" Ref="R7"  Part="1"
 AR Path="/597E1B39/589BE76D" Ref="R5"  Part="1"
-F 0 "R9" V 4480 3950 50  0000 C CNN
+AR Path="/589BE76D" Ref="R?"  Part="1"
+F 0 "R11" V 4480 3950 50  0000 C CNN
 F 1 "100" V 4400 3950 50  0000 C CNN
 F 2 "Resistor_SMD:R_0603_1608Metric" V 4330 3950 50  0001 C CNN
@@
 IR_LED
 $Comp
-L power:GND #PWR037
+L KERISE-rescue:GND-power-KERISE-rescue-KERISE-rescue #PWR036
 U 1 1 589BF265
 P 4400 3000
-AR Path="/57CF0B09/589BF265" Ref="#PWR037"  Part="1"
-AR Path="/57CF2A30/589BF265" Ref="#PWR035"  Part="1"
-AR Path="/597E1B35/589BF265" Ref="#PWR028"  Part="1"
-AR Path="/597E1B39/589BF265" Ref="#PWR026"  Part="1"
-F 0 "#PWR035" H 4400 2750 50  0001 C CNN
+AR Path="/57CF0B09/589BF265" Ref="#PWR036"  Part="1"
+AR Path="/57CF2A30/589BF265" Ref="#PWR034"  Part="1"
+AR Path="/597E1B35/589BF265" Ref="#PWR027"  Part="1"
+AR Path="/597E1B39/589BF265" Ref="#PWR025"  Part="1"
+AR Path="/589BF265" Ref="#PWR?"  Part="1"
+F 0 "#PWR036" H 4400 2750 50  0001 C CNN
 F 1 "GND" H 4400 2850 50  0000 C CNN
 F 2 "" H 4400 3000 50  0000 C CNN
@@
 	4400 5200 4400 5500
 $Comp
-L Device:LED D8
+L KERISE-rescue:LED-Device-KERISE-rescue-KERISE-rescue D8
 U 1 1 594AC674
 P 4400 4450
@@
 AR Path="/597E1B35/594AC674" Ref="D6"  Part="1"
 AR Path="/597E1B39/594AC674" Ref="D5"  Part="1"
-F 0 "D7" V 4500 4300 50  0000 C CNN
+AR Path="/594AC674" Ref="D?"  Part="1"
+F 0 "D8" V 4500 4300 50  0000 C CNN
 F 1 "SFH4045N" V 4400 4150 50  0000 C CNN
 F 2 "mouse:SFH4045N_L" H 4400 4450 50  0001 C CNN
@@
 $EndComp
 $Comp
-L power:+3.3V #PWR036
+L KERISE-rescue:+3.3V-power-KERISE-rescue-KERISE-rescue #PWR035
 U 1 1 5A172FEF
 P 4400 2500
-AR Path="/57CF0B09/5A172FEF" Ref="#PWR036"  Part="1"
-AR Path="/57CF2A30/5A172FEF" Ref="#PWR034"  Part="1"
-AR Path="/597E1B35/5A172FEF" Ref="#PWR027"  Part="1"
-AR Path="/597E1B39/5A172FEF" Ref="#PWR025"  Part="1"
-F 0 "#PWR034" H 4400 2350 50  0001 C CNN
+AR Path="/57CF0B09/5A172FEF" Ref="#PWR035"  Part="1"
+AR Path="/57CF2A30/5A172FEF" Ref="#PWR033"  Part="1"
+AR Path="/597E1B35/5A172FEF" Ref="#PWR026"  Part="1"
+AR Path="/597E1B39/5A172FEF" Ref="#PWR024"  Part="1"
+AR Path="/5A172FEF" Ref="#PWR?"  Part="1"
+F 0 "#PWR035" H 4400 2350 50  0001 C CNN
 F 1 "+3.3V" H 4400 2640 50  0000 C CNN
 F 2 "" H 4400 2500 50  0001 C CNN
@@
 	5300 2900 5200 2900
 $Comp
-L Device:C C16
+L KERISE-rescue:C-Device-KERISE-rescue-KERISE-rescue C16
 U 1 1 5A1B992B
 P 5000 5050
@@
 AR Path="/597E1B35/5A1B992B" Ref="C10"  Part="1"
 AR Path="/597E1B39/5A1B992B" Ref="C8"  Part="1"
-F 0 "C14" H 5025 5150 50  0000 L CNN
+AR Path="/5A1B992B" Ref="C?"  Part="1"
+F 0 "C16" H 5025 5150 50  0000 L CNN
 F 1 "1u" H 5025 4950 50  0000 L CNN
 F 2 "Capacitor_SMD:C_0402_1005Metric" H 5038 4900 50  0001 C CNN
@@
 $EndComp
 $Comp
-L Device:Q_Photo_NPN Q9
+L KERISE-rescue:Q_Photo_NPN-Device-KERISE-rescue-KERISE-rescue Q9
 U 1 1 5A4ADF8B
 P 5500 4500
@@
 AR Path="/597E1B35/5A4ADF8B" Ref="Q5"  Part="1"
 AR Path="/597E1B39/5A4ADF8B" Ref="Q3"  Part="1"
-F 0 "Q7" H 5700 4550 50  0000 L CNN
+AR Path="/5A4ADF8B" Ref="Q?"  Part="1"
+F 0 "Q9" H 5700 4550 50  0000 L CNN
 F 1 "SFH3015FA" H 5700 4450 50  0000 L CNN
 F 2 "mouse:SFH3015FA_L" H 5700 4600 50  0001 C CNN
@@
 $EndComp
 $Comp
-L Device:R R12
+L KERISE-rescue:R-Device-KERISE-rescue-KERISE-rescue R12
 U 1 1 589BEE3B
 P 5600 5050
@@
 AR Path="/597E1B35/589BEE3B" Ref="R8"  Part="1"
 AR Path="/597E1B39/589BEE3B" Ref="R6"  Part="1"
-F 0 "R10" V 5680 5050 50  0000 C CNN
+AR Path="/589BEE3B" Ref="R?"  Part="1"
+F 0 "R12" V 5680 5050 50  0000 C CNN
 F 1 "10k" V 5600 5050 50  0000 C CNN
 F 2 "Resistor_SMD:R_0201_0603Metric" V 5530 5050 50  0001 C CNN
@@
 	5600 4900 5600 4800
 $Comp
-L Device:C_Small C15
+L KERISE-rescue:C_Small-Device-KERISE-rescue-KERISE-rescue C15
 U 1 1 5C29B79F
 P 6600 4800
@@
 AR Path="/597E1B35/5C29B79F" Ref="C11"  Part="1"
 AR Path="/597E1B39/5C29B79F" Ref="C9"  Part="1"
-F 0 "C15" H 6692 4846 50  0000 L CNN
+AR Path="/5C29B79F" Ref="C?"  Part="1"
+F 0 "C17" H 6692 4846 50  0000 L CNN
 F 1 "0.1u" H 6692 4755 50  0000 L CNN
 F 2 "Capacitor_SMD:C_0201_0603Metric" H 6600 4800 50  0001 C CNN
@@
 s_3.3V
 $Comp
-L Connector:Conn_01x04_Female J12
+L KERISE-rescue:Conn_01x04_Female-Connector-KERISE-rescue-KERISE-rescue J12
 U 1 1 5E4BA6B8
 P 4700 2700
@@
 AR Path="/597E1B35/5E4BA6B8" Ref="J3"  Part="1"
 AR Path="/597E1B39/5E4BA6B8" Ref="J1"  Part="1"
-F 0 "J10" H 4728 2676 50  0000 L CNN
+AR Path="/5E4BA6B8" Ref="J?"  Part="1"
+F 0 "J12" H 4728 2676 50  0000 L CNN
 F 1 "Host" H 4728 2585 50  0000 L CNN
 F 2 "mouse:IR_HOST_V_04" H 4700 2700 50  0001 C CNN
@@
 $EndComp
 $Comp
-L Connector:Conn_01x04_Male J13
+L KERISE-rescue:Conn_01x04_Male-Connector-KERISE-rescue-KERISE-rescue J13
 U 1 1 5E4BAD76
 P 5000 2700
@@
 AR Path="/597E1B35/5E4BAD76" Ref="J4"  Part="1"
 AR Path="/597E1B39/5E4BAD76" Ref="J2"  Part="1"
-F 0 "J11" H 5108 2981 50  0000 C CNN
+AR Path="/5E4BAD76" Ref="J?"  Part="1"
+F 0 "J13" H 5108 2981 50  0000 C CNN
 F 1 "Slave" H 5108 2890 50  0000 C CNN
 F 2 "mouse:IR_SLAVE_V_04" H 5000 2700 50  0001 C CNN
