File: kicad/COM.sch (KiCad schematic (older format))
At the start: 1 part, among them J7 COM

Commit message: 予備配線完了
Parts:
- renumbered J7 to J9
Changed lines of the file:
@@
 $EndDescr
 $Comp
-L power:GND #PWR039
+L power:GND #PWR033
 U 1 1 57CDAC76
 P 4800 4200
-F 0 "#PWR039" H 4800 3950 50  0001 C CNN
+F 0 "#PWR033" H 4800 3950 50  0001 C CNN
 F 1 "GND" H 4800 4050 50  0000 C CNN
 F 2 "" H 4800 4200 50  0000 C CNN
@@
 COM Port
 $Comp
-L Connector:Conn_01x03_Male J7
+L Connector:Conn_01x03_Male J9
 U 1 1 5B6F3423
 P 4500 4000
-F 0 "J7" H 4606 4278 50  0000 C CNN
+F 0 "J9" H 4606 4278 50  0000 C CNN
 F 1 "COM" H 4606 4187 50  0000 C CNN
 F 2 "mouse:JST_SH_BM03B-SRSS-TB_03x1.00mm_Straight" H 4500 4000 50  0001 C CNN

Commit message: KiCad: update pcb
Parts:
- J9: symbol Connector:Conn_01x03_Male -> KERISE-rescue:Conn_01x03_Male-Connector-KERISE-rescue-KERISE-rescue
Changed lines of the file:
@@
 $Descr A4 11693 8268
 encoding utf-8
-Sheet 6 13
+Sheet 9 13
 Title ""
 Date ""
@@
 $EndDescr
 $Comp
-L power:GND #PWR033
+L KERISE-rescue:GND-power-KERISE-rescue-KERISE-rescue #PWR032
 U 1 1 57CDAC76
 P 4800 4200
-F 0 "#PWR033" H 4800 3950 50  0001 C CNN
+F 0 "#PWR032" H 4800 3950 50  0001 C CNN
 F 1 "GND" H 4800 4050 50  0000 C CNN
 F 2 "" H 4800 4200 50  0000 C CNN
@@
 COM Port
 $Comp
-L Connector:Conn_01x03_Male J9
+L KERISE-rescue:Conn_01x03_Male-Connector-KERISE-rescue-KERISE-rescue J9
 U 1 1 5B6F3423
 P 4500 4000
