File: kicad/IMU.sch (KiCad schematic (older format))
At the start: 3 parts, among them U6 ICM-20602

Commit message: 予備配線完了
Parts:
- renumbered C18 to C6, C19 to C7, U6 to U4
Changed lines of the file:
@@
 P 5600 3400
 AR Path="/57CC33F6/592C611A" Ref="U?"  Part="1"
-AR Path="/5A18D4D6/592C611A" Ref="U6"  Part="1"
-F 0 "U6" H 5600 4150 60  0000 C CNN
+AR Path="/5A18D4D6/592C611A" Ref="U4"  Part="1"
+F 0 "U4" H 5600 4150 60  0000 C CNN
 F 1 "ICM-20602" H 5600 4000 60  0000 C CNN
 F 2 "mouse:ICM-20602" H 5600 4000 60  0001 C CNN
@@
 P 4800 3700
 AR Path="/57CC33F6/592C613A" Ref="C?"  Part="1"
-AR Path="/5A18D4D6/592C613A" Ref="C19"  Part="1"
-F 0 "C19" H 4810 3770 50  0000 L CNN
+AR Path="/5A18D4D6/592C613A" Ref="C7"  Part="1"
+F 0 "C7" H 4810 3770 50  0000 L CNN
 F 1 "0.1u" H 4810 3620 50  0000 L CNN
 F 2 "Capacitor_SMD:C_0201_0603Metric" H 4800 3700 50  0001 C CNN
@@
 P 4600 3700
 AR Path="/57CC33F6/592C6186" Ref="C?"  Part="1"
-AR Path="/5A18D4D6/592C6186" Ref="C18"  Part="1"
-F 0 "C18" H 4610 3770 50  0000 L CNN
+AR Path="/5A18D4D6/592C6186" Ref="C6"  Part="1"
+F 0 "C6" H 4610 3770 50  0000 L CNN
 F 1 "0.1u" H 4610 3620 50  0000 L CNN
 F 2 "Capacitor_SMD:C_0201_0603Metric" H 4600 3700 50  0001 C CNN
@@
 P 5000 4200
 AR Path="/57CC33F6/592C63E1" Ref="#PWR?"  Part="1"
-AR Path="/5A18D4D6/592C63E1" Ref="#PWR051"  Part="1"
-F 0 "#PWR051" H 5000 3950 50  0001 C CNN
+AR Path="/5A18D4D6/592C63E1" Ref="#PWR023"  Part="1"
+F 0 "#PWR023" H 5000 3950 50  0001 C CNN
 F 1 "GND" H 5000 4050 50  0000 C CNN
 F 2 "" H 5000 4200 50  0000 C CNN
@@
 P 4800 4200
 AR Path="/57CC33F6/592C640D" Ref="#PWR?"  Part="1"
-AR Path="/5A18D4D6/592C640D" Ref="#PWR049"  Part="1"
-F 0 "#PWR049" H 4800 3950 50  0001 C CNN
+AR Path="/5A18D4D6/592C640D" Ref="#PWR021"  Part="1"
+F 0 "#PWR021" H 4800 3950 50  0001 C CNN
 F 1 "GND" H 4800 4050 50  0000 C CNN
 F 2 "" H 4800 4200 50  0000 C CNN
@@
 P 4600 4200
 AR Path="/57CC33F6/592C6444" Ref="#PWR?"  Part="1"
-AR Path="/5A18D4D6/592C6444" Ref="#PWR048"  Part="1"
-F 0 "#PWR048" H 4600 3950 50  0001 C CNN
+AR Path="/5A18D4D6/592C6444" Ref="#PWR020"  Part="1"
+F 0 "#PWR020" H 4600 3950 50  0001 C CNN
 F 1 "GND" H 4600 4050 50  0000 C CNN
 F 2 "" H 4600 4200 50  0000 C CNN
@@
 P 5000 2800
 AR Path="/57CC33F6/592C64FB" Ref="#PWR?"  Part="1"
-AR Path="/5A18D4D6/592C64FB" Ref="#PWR050"  Part="1"
-F 0 "#PWR050" H 5000 2650 50  0001 C CNN
+AR Path="/5A18D4D6/592C64FB" Ref="#PWR022"  Part="1"
+F 0 "#PWR022" H 5000 2650 50  0001 C CNN
 F 1 "+3.3V" H 5000 2940 50  0000 C CNN
 F 2 "" H 5000 2800 50  0000 C CNN
@@
 P 6200 3500
 AR Path="/57CC33F6/592C6B85" Ref="#PWR?"  Part="1"
-AR Path="/5A18D4D6/592C6B85" Ref="#PWR052"  Part="1"
-F 0 "#PWR052" H 6200 3250 50  0001 C CNN
+AR Path="/5A18D4D6/592C6B85" Ref="#PWR024"  Part="1"
+F 0 "#PWR024" H 6200 3250 50  0001 C CNN
 F 1 "GND" H 6200 3350 50  0000 C CNN
 F 2 "" H 6200 3500 50  0000 C CNN

Commit message: update kicad .gitignore
Other:
- note added: "IMU"
- note removed: "AXIS Sensor"
Changed lines of the file:
@@
 $Descr A4 11693 8268
 encoding utf-8
-Sheet 11 13
+Sheet 4 13
 Title ""
 Date ""
@@
 Comment4 ""
 $EndDescr
-Text Notes 4200 2400 0    100  ~ 0
-AXIS Sensor
+Text Notes 4500 2500 0    100  ~ 0
+IMU
 $Comp
 L KERISE:ICM-20602 U?

Commit message: KiCad: update pcb
Parts:
- removed U4: ICM-20602, mouse:ICM-20602, symbol KERISE:ICM-20602
- added U4: ICM-20600, mouse:ICM-20600, symbol KERISE:ICM-20600
- C6, C7: symbol Device:C_Small -> KERISE-rescue:C_Small-Device-KERISE-rescue-KERISE-rescue
Connections:
- net +3V3: now also U4.5 (VDDIO), U4.8 (VDD)
- net CS: now also U4.12 (~CS)
- net GND: now also U4.6 (GND), U4.7 (RESV)
- net MISO: now also U4.1 (SA0/SDO)
- net MOSI: now also U4.14 (SDA/SDI)
- net SCLK: now also U4.13 (SCL/SCLK)
- net at C7.1: now also U4.11 (REGOUT)
- no-connect marks 1 -> 3
Changed lines of the file:
@@
 IMU
 $Comp
-L KERISE:ICM-20602 U?
-U 1 1 592C611A
-P 5600 3400
-AR Path="/57CC33F6/592C611A" Ref="U?"  Part="1"
-AR Path="/5A18D4D6/592C611A" Ref="U4"  Part="1"
-F 0 "U4" H 5600 4150 60  0000 C CNN
-F 1 "ICM-20602" H 5600 4000 60  0000 C CNN
-F 2 "mouse:ICM-20602" H 5600 4000 60  0001 C CNN
-F 3 "" H 5600 4000 60  0000 C CNN
-	1    5600 3400
-	1    0    0    -1
-$EndComp
-$Comp
-L Device:C_Small C?
+L KERISE-rescue:C_Small-Device-KERISE-rescue-KERISE-rescue C?
 U 1 1 592C613A
 P 4800 3700
 AR Path="/57CC33F6/592C613A" Ref="C?"  Part="1"
 AR Path="/5A18D4D6/592C613A" Ref="C7"  Part="1"
+AR Path="/592C613A" Ref="C?"  Part="1"
 F 0 "C7" H 4810 3770 50  0000 L CNN
 F 1 "0.1u" H 4810 3620 50  0000 L CNN
@@
 $EndComp
 $Comp
-L Device:C_Small C?
+L KERISE-rescue:C_Small-Device-KERISE-rescue-KERISE-rescue C?
 U 1 1 592C6186
 P 4600 3700
 AR Path="/57CC33F6/592C6186" Ref="C?"  Part="1"
 AR Path="/5A18D4D6/592C6186" Ref="C6"  Part="1"
+AR Path="/592C6186" Ref="C?"  Part="1"
 F 0 "C6" H 4610 3770 50  0000 L CNN
 F 1 "0.1u" H 4610 3620 50  0000 L CNN
@@
 $EndComp
 $Comp
-L power:GND #PWR?
+L KERISE-rescue:GND-power-KERISE-rescue-KERISE-rescue #PWR?
 U 1 1 592C63E1
 P 5000 4200
 AR Path="/57CC33F6/592C63E1" Ref="#PWR?"  Part="1"
 AR Path="/5A18D4D6/592C63E1" Ref="#PWR023"  Part="1"
+AR Path="/592C63E1" Ref="#PWR?"  Part="1"
 F 0 "#PWR023" H 5000 3950 50  0001 C CNN
 F 1 "GND" H 5000 4050 50  0000 C CNN
@@
 $EndComp
 $Comp
-L power:GND #PWR?
+L KERISE-rescue:GND-power-KERISE-rescue-KERISE-rescue #PWR?
 U 1 1 592C640D
 P 4800 4200
 AR Path="/57CC33F6/592C640D" Ref="#PWR?"  Part="1"
 AR Path="/5A18D4D6/592C640D" Ref="#PWR021"  Part="1"
+AR Path="/592C640D" Ref="#PWR?"  Part="1"
 F 0 "#PWR021" H 4800 3950 50  0001 C CNN
 F 1 "GND" H 4800 4050 50  0000 C CNN
@@
 $EndComp
 $Comp
-L power:GND #PWR?
+L KERISE-rescue:GND-power-KERISE-rescue-KERISE-rescue #PWR?
 U 1 1 592C6444
 P 4600 4200
 AR Path="/57CC33F6/592C6444" Ref="#PWR?"  Part="1"
 AR Path="/5A18D4D6/592C6444" Ref="#PWR020"  Part="1"
+AR Path="/592C6444" Ref="#PWR?"  Part="1"
 F 0 "#PWR020" H 4600 3950 50  0001 C CNN
 F 1 "GND" H 4600 4050 50  0000 C CNN
@@
 $EndComp
 $Comp
-L power:+3.3V #PWR?
+L KERISE-rescue:+3.3V-power-KERISE-rescue-KERISE-rescue #PWR?
 U 1 1 592C64FB
 P 5000 2800
 AR Path="/57CC33F6/592C64FB" Ref="#PWR?"  Part="1"
 AR Path="/5A18D4D6/592C64FB" Ref="#PWR022"  Part="1"
+AR Path="/592C64FB" Ref="#PWR?"  Part="1"
 F 0 "#PWR022" H 5000 2650 50  0001 C CNN
 F 1 "+3.3V" H 5000 2940 50  0000 C CNN
@@
 MISO
 NoConn ~ 6100 3300
-$Comp
-L power:GND #PWR?
-U 1 1 592C6B85
-P 6200 3500
-AR Path="/57CC33F6/592C6B85" Ref="#PWR?"  Part="1"
-AR Path="/5A18D4D6/592C6B85" Ref="#PWR024"  Part="1"
-F 0 "#PWR024" H 6200 3250 50  0001 C CNN
-F 1 "GND" H 6200 3350 50  0000 C CNN
-F 2 "" H 6200 3500 50  0000 C CNN
-F 3 "" H 6200 3500 50  0000 C CNN
-	1    6200 3500
-	1    0    0    -1
-$EndComp
 Text HLabel 6100 3000 2    60   Input ~ 0
 MOSI
@@
 	4800 4200 4800 3800
 Connection ~ 5000 4100
-Connection ~ 5000 3600
-Wire Wire Line
-	5000 3500 5100 3500
-Connection ~ 5000 3700
 Wire Wire Line
 	5000 3600 5100 3600
-Connection ~ 5000 3800
-Wire Wire Line
-	5000 3700 5100 3700
-Connection ~ 5000 3900
-Wire Wire Line
-	5100 3800 5000 3800
-Wire Wire Line
-	5000 3900 5100 3900
-Wire Wire Line
-	5000 3500 5000 3600
 Wire Wire Line
 	5000 4100 5100 4100
 Wire Wire Line
 	4600 3000 4600 3600
-Wire Wire Line
-	6100 3400 6200 3400
-Wire Wire Line
-	6200 3400 6200 3500
 Connection ~ 5000 2900
 Wire Wire Line
@@
 	5000 4100 5000 4200
 Wire Wire Line
-	5000 3600 5000 3700
-Wire Wire Line
-	5000 3700 5000 3800
-Wire Wire Line
-	5000 3800 5000 3900
-Wire Wire Line
-	5000 3900 5000 4100
-Wire Wire Line
 	5000 2900 5000 3000
 Wire Wire Line
 	5000 3000 5100 3000
+$Comp
+L KERISE:ICM-20600 U4
+U 1 1 61998ECC
+P 5600 3400
+F 0 "U4" H 5600 4287 60  0000 C CNN
+F 1 "ICM-20600" H 5600 4181 60  0000 C CNN
+F 2 "mouse:ICM-20600" H 5600 4000 60  0001 C CNN
+F 3 "" H 5600 4000 60  0000 C CNN
+	1    5600 3400
+	1    0    0    -1
+$EndComp
+Wire Wire Line
+	5000 3600 5000 4100
+NoConn ~ 6100 3400
+NoConn ~ 6100 3500
 $EndSCHEMATC
