File: kicad/KERISE.kicad_pcb (KiCad board)
At the start: 2 copper layers, 40.5 x 38.8 mm, 90 parts, among them J1 Host, J10 Host, J11 Slave, J12 Host, J13 Slave, J14 Motor_L, J15 Motor_R, J2 Slave, J3 Host, J4 Slave, J5 ENC_Host, J6 ENC_Slave, J7 ENC_Host, J8 ENC_Slave, J9 COM, P1 ToF_Host, P2 ToF_Slave, Q1 DMN3065LW-7, Q2 DMN3065LW-7, Q3 SFH3015FA, Q4 DMN3065LW-7, Q5 SFH3015FA, Q6 DMN3065LW-7, Q7 SFH3015FA, Q8 DMN3065LW-7, Q9 SFH3015FA, SW1 RESET, SW2 UPLOAD, U1 ESP32-PICO-D4, U2 VL6180X, U3 PCA9632, U4 ICM-20602, U5 MA730, U6 MA730, U7 LXDC2UR30, U8 DRV8835

Commit message: 自動配線を適用
Parts:
- added G***: LOGO, mouse:KERI_9mm, B.Cu at (148.5, 114.0)
Routing:
- net +3V3: track 4.24 -> 114.9 mm, vias 0 -> 2
- net GND: track 35.3 -> 144.9 mm, vias 0 -> 4
- net PR-RCV-FR: track 0.00 -> 64.3 mm, vias 0 -> 2
- net SPI-MOSI: track 0.00 -> 42.6 mm, vias 0 -> 2
- net SPI-SCLK: track 0.00 -> 36.4 mm, vias 0 -> 3
- net SPI-MISO: track 0.00 -> 32.4 mm, vias 0 -> 3
- net Net-(D4-Pad1): track 0.00 -> 30.2 mm, vias 0 -> 2
- net I2C-SDA: track 0.00 -> 28.0 mm, vias 0 -> 2
- net SPI-CS-ENC_L: track 0.00 -> 27.0 mm, vias 0 -> 2
- net PR-RCV-SR: track 0.00 -> 25.2 mm, vias 0 -> 2
- net UART-TX: track 0.00 -> 23.9 mm, vias 0 -> 2
- net UART-RX: track 0.00 -> 23.6 mm, vias 0 -> 2
- net I2C-SCL: track 0.00 -> 23.5 mm, vias 0 -> 2
- net BUTTON: track 0.00 -> 22.2 mm, vias 0 -> 2
- net PR-LED-FL: track 0.00 -> 20.6 mm, vias 0 -> 2
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Other:
- board text added: "2020.03.20"
- board text removed: "2020.02.20"

Commit message: KiCad: update pcb
Parts:
- C10, C14, C16, C8: value 2.2u -> 1u
- LS1: footprint mouse:SMT-0440-S-R -> mouse:SMT-0340-T-R
- U4: value ICM-20602 -> ICM-20600; footprint mouse:ICM-20602 -> mouse:ICM-20600
- U5, U6: footprint mouse:QFN-16-1EP_3x3mm_P0.5mm -> mouse:MA730
- moved C6 5.00 mm to (146.5, 113.0), turned to 90 degrees
- moved C4 2.24 mm to (158.5, 105.5)
- moved R2 1.25 mm to (168.8, 131.5)
- moved R3 1.25 mm to (170.2, 131.5)
- moved C3 1.00 mm to (169.5, 130.5)
- moved G*** 1.00 mm to (148.5, 113.0)
- moved U2 1.00 mm to (169.5, 128.5)
- moved C21 0.50 mm to (146.0, 116.5)
- moved R14 0.25 mm to (146.0, 115.2)
- moved C19 0.10 mm to (151.5, 101.4)
- moved C20 0.10 mm to (145.5, 101.4), turned to 270 degrees
- turned J1 to 170 degrees
- turned J10 to 125 degrees
- turned J12 to 235 degrees
- turned J3 to 190 degrees
Connections:
- U4 pad 1: +3V3 -> SPI-MISO
- U4 pad 11: GND -> Net-(C7-Pad1)
- U4 pad 12: GND -> SPI-CS-IMU
- U4 pad 13: GND -> SPI-SCLK
- U4 pad 14: Net-(C7-Pad1) -> SPI-MOSI
- U4 pad 4: SPI-MISO -> (no net)
- U4 pad 5: SPI-CS-IMU -> +3V3
- U4 pad 6: (no net) -> GND
- U4 pad 8: GND -> +3V3
Routing:
- net +3V3: track 114.9 -> 131.8 mm
- net I2C-SCL: track 23.5 -> 31.9 mm, vias 2 -> 4
- net PR-RCV-SL: track 12.4 -> 20.6 mm, vias 0 -> 2
- net GND: track 144.9 -> 152.1 mm
- net /ToF/s_3.3V: track 12.5 -> 14.5 mm
- net SPI-SCLK: track 36.4 -> 38.4 mm
- net Net-(D2-Pad1): track 11.9 -> 9.92 mm
- net PR-RCV-FL: track 9.79 -> 11.5 mm
- net SPI-MOSI: track 42.6 -> 44.1 mm
- net I2C-SDA: track 28.0 -> 26.6 mm, vias 2 -> 4
- net Net-(C7-Pad1): track 2.39 -> 1.02 mm
- net PR-LED-FR: track 15.8 -> 17.0 mm
- net Net-(D3-Pad1): track 18.4 -> 19.5 mm
- net /ToF/s_SCL: track 3.77 -> 4.81 mm
- net SPI-MISO: track 32.4 -> 33.4 mm
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Other:
- outline, holes or cut-outs redrawn
- board text added: "2021.11.20"
- board text added: "KERISE v5.2"
- board text removed: "2020.03.20"
- board text removed: "KERISE v5"
