File: kicad/KERISE.kicad_pcb (KiCad board)
At the start: 2 copper layers, 40.5 x 38.8 mm, 91 parts, among them J1 Host, J10 Host, J11 Slave, J12 Host, J13 Slave, J14 Motor_L, J15 Motor_R, J2 Slave, J3 Host, J4 Slave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

Commit message: update to kicad 7
Other:
- net class 3.3V removed
- net class Analog removed
- net class Antena removed
- net class BATT removed
- net class Default removed
- net class GND removed
- net class LED removed
- net class Motor removed
