File: kicad/KERISE.sch (KiCad schematic (older format))
At the start: 5 parts, among them SW1 RESET, U1 ESP32-PICO-D4

Commit message: 予備配線完了
Parts:
- removed AE1: Antenna, mouse:HIDDEN_PAD, symbol Device:Antenna
Connections:
- net ANTENA: no longer names the net of U1.2 (LNA_IN)
- no-connect marks 14 -> 15

Commit message: KiCad: update pcb
Parts:
- C1: symbol Device:C_Small -> KERISE-rescue:C_Small-Device-KERISE-rescue-KERISE-rescue
- R1: symbol Device:R_Small -> KERISE-rescue:R_Small-Device-KERISE-rescue-KERISE-rescue
- SW1: symbol Switch:SW_Push -> KERISE-rescue:SW_Push-Switch-KERISE-rescue-KERISE-rescue
Changed lines of the file:
@@
 BUTTON
 $Comp
-L power:GND #PWR05
+L KERISE-rescue:GND-power-KERISE-rescue-KERISE-rescue #PWR05
 U 1 1 58964ED8
 P 10300 3400
@@
 UART-RX
 $Comp
-L power:+3.3V #PWR03
+L KERISE-rescue:+3.3V-power-KERISE-rescue-KERISE-rescue #PWR03
 U 1 1 58A4281C
 P 10100 2900
@@
 $EndComp
 $Comp
-L Device:R_Small R1
+L KERISE-rescue:R_Small-Device-KERISE-rescue-KERISE-rescue R1
 U 1 1 58A7844B
 P 9900 3000
@@
 NoConn ~ 5600 4300
 $Comp
-L power:GND #PWR04
+L KERISE-rescue:GND-power-KERISE-rescue-KERISE-rescue #PWR04
 U 1 1 58A70C45
 P 10200 2300
@@
 $EndComp
 $Comp
-L Device:C_Small C1
+L KERISE-rescue:C_Small-Device-KERISE-rescue-KERISE-rescue C1
 U 1 1 58A9401A
 P 10000 1000
@@
 	9700 1400 9700 1200
 $Comp
-L Switch:SW_Push SW1
+L KERISE-rescue:SW_Push-Switch-KERISE-rescue-KERISE-rescue SW1
 U 1 1 5B6F20EF
 P 10000 3300
@@
 $EndComp
 $Comp
-L power:GND #PWR02
+L KERISE-rescue:GND-power-KERISE-rescue-KERISE-rescue #PWR02
 U 1 1 5B709AF6
 P 9700 5000
@@
 $EndComp
 $Comp
-L power:+3.3V #PWR01
+L KERISE-rescue:+3.3V-power-KERISE-rescue-KERISE-rescue #PWR01
 U 1 1 5B709B26
 P 9700 900
