File: kicad/Motor.sch (KiCad schematic (older format))
At the start: 8 parts, among them J1 Motor_L, J2 Motor_R, U2 DRV8835

Commit message: 予備配線完了
Parts:
- renumbered C2 to C21, C3 to C22, C4 to C23, J1 to J14, J2 to J15, U2 to U8
Changed lines of the file:
@@
 $EndDescr
 $Comp
-L KERISE:DRV8835 U2
+L KERISE:DRV8835 U8
 U 1 1 57CA1E0F
 P 5500 3600
-F 0 "U2" H 5050 3950 60  0000 L CNN
+F 0 "U8" H 5050 3950 60  0000 L CNN
 F 1 "DRV8835" H 5650 3950 60  0000 L CNN
 F 2 "mouse:DRV8835" H 5100 3750 60  0001 C CNN
@@
 $EndComp
 $Comp
-L power:GND #PWR012
+L power:GND #PWR062
 U 1 1 57CA1E46
 P 4800 4200
-F 0 "#PWR012" H 4800 3950 50  0001 C CNN
+F 0 "#PWR062" H 4800 3950 50  0001 C CNN
 F 1 "GND" H 4800 4050 50  0000 C CNN
 F 2 "" H 4800 4200 50  0000 C CNN
@@
 Motor
 $Comp
-L Device:C C4
+L Device:C C23
 U 1 1 57CCEFE0
 P 4000 3650
-F 0 "C4" H 4025 3750 50  0000 L CNN
+F 0 "C23" H 4025 3750 50  0000 L CNN
 F 1 "0.1u" H 4025 3550 50  0000 L CNN
 F 2 "Capacitor_SMD:C_0201_0603Metric" H 4038 3500 50  0001 C CNN
@@
 $EndComp
 $Comp
-L power:+BATT #PWR015
+L power:+BATT #PWR065
 U 1 1 57CD5BEE
 P 5600 3100
-F 0 "#PWR015" H 5600 2950 50  0001 C CNN
+F 0 "#PWR065" H 5600 2950 50  0001 C CNN
 F 1 "+BATT" H 5600 3240 50  0000 C CNN
 F 2 "" H 5600 3100 50  0000 C CNN
@@
 MT_OUT_R2
 $Comp
-L power:+3.3V #PWR013
+L power:+3.3V #PWR063
 U 1 1 589CC6A5
 P 5300 3100
-F 0 "#PWR013" H 5300 2950 50  0001 C CNN
+F 0 "#PWR063" H 5300 2950 50  0001 C CNN
 F 1 "+3.3V" H 5300 3240 50  0000 C CNN
 F 2 "" H 5300 3100 50  0000 C CNN
@@
 $EndComp
 $Comp
-L power:+3.3V #PWR010
+L power:+3.3V #PWR060
 U 1 1 589CC6C6
 P 4000 3100
-F 0 "#PWR010" H 4000 2950 50  0001 C CNN
+F 0 "#PWR060" H 4000 2950 50  0001 C CNN
 F 1 "+3.3V" H 4000 3240 50  0000 C CNN
 F 2 "" H 4000 3100 50  0000 C CNN
@@
 $EndComp
 $Comp
-L power:+BATT #PWR08
+L power:+BATT #PWR058
 U 1 1 594721DF
 P 3700 3100
-F 0 "#PWR08" H 3700 2950 50  0001 C CNN
+F 0 "#PWR058" H 3700 2950 50  0001 C CNN
 F 1 "+BATT" H 3700 3240 50  0000 C CNN
 F 2 "" H 3700 3100 50  0000 C CNN
@@
 $EndComp
 $Comp
-L Device:C C3
+L Device:C C22
 U 1 1 594721FA
 P 3700 3650
-F 0 "C3" H 3725 3750 50  0000 L CNN
+F 0 "C22" H 3725 3750 50  0000 L CNN
 F 1 "0.1u" H 3725 3550 50  0000 L CNN
 F 2 "Capacitor_SMD:C_0201_0603Metric" H 3738 3500 50  0001 C CNN
@@
 MT_OUT_L_R
 $Comp
-L Connector_Generic:Conn_01x02 J1
+L Connector_Generic:Conn_01x02 J14
 U 1 1 5B6F504A
 P 8400 3400
-F 0 "J1" H 8479 3392 50  0000 L CNN
+F 0 "J14" H 8479 3392 50  0000 L CNN
 F 1 "Motor_L" H 8479 3301 50  0000 L CNN
 F 2 "mouse:SMD_conn_2" H 8400 3400 50  0001 C CNN
@@
 $EndComp
 $Comp
-L Connector_Generic:Conn_01x02 J2
+L Connector_Generic:Conn_01x02 J15
 U 1 1 5B6F50A6
 P 8400 3900
-F 0 "J2" H 8480 3892 50  0000 L CNN
+F 0 "J15" H 8480 3892 50  0000 L CNN
 F 1 "Motor_R" H 8480 3801 50  0000 L CNN
 F 2 "mouse:SMD_conn_2" H 8400 3900 50  0001 C CNN
@@
 $EndComp
 $Comp
-L power:GND #PWR016
+L power:GND #PWR066
 U 1 1 5B6FD311
 P 5700 4200
-F 0 "#PWR016" H 5700 3950 50  0001 C CNN
+F 0 "#PWR066" H 5700 3950 50  0001 C CNN
 F 1 "GND" H 5700 4050 50  0000 C CNN
 F 2 "" H 5700 4200 50  0000 C CNN
@@
 $EndComp
 $Comp
-L power:GND #PWR011
+L power:GND #PWR061
 U 1 1 5B6FD364
 P 4000 4200
-F 0 "#PWR011" H 4000 3950 50  0001 C CNN
+F 0 "#PWR061" H 4000 3950 50  0001 C CNN
 F 1 "GND" H 4000 4050 50  0000 C CNN
 F 2 "" H 4000 4200 50  0000 C CNN
@@
 $EndComp
 $Comp
-L power:GND #PWR09
+L power:GND #PWR059
 U 1 1 5B7097B0
 P 3700 4200
-F 0 "#PWR09" H 3700 3950 50  0001 C CNN
+F 0 "#PWR059" H 3700 3950 50  0001 C CNN
 F 1 "GND" H 3700 4050 50  0000 C CNN
 F 2 "" H 3700 4200 50  0000 C CNN
@@
 $EndComp
 $Comp
-L power:GND #PWR014
+L power:GND #PWR064
 U 1 1 5B7097C9
 P 5400 4200
-F 0 "#PWR014" H 5400 3950 50  0001 C CNN
+F 0 "#PWR064" H 5400 3950 50  0001 C CNN
 F 1 "GND" H 5400 4050 50  0000 C CNN
 F 2 "" H 5400 4200 50  0000 C CNN
@@
 $EndComp
 $Comp
-L Device:C C2
+L Device:C C21
 U 1 1 5C29DB96
 P 3300 3650
-F 0 "C2" H 3415 3696 50  0000 L CNN
+F 0 "C21" H 3415 3696 50  0000 L CNN
 F 1 "47u" H 3415 3605 50  0000 L CNN
 F 2 "Capacitor_SMD:C_0805_2012Metric" H 3338 3500 50  0001 C CNN
@@
 $EndComp
 $Comp
-L power:GND #PWR07
+L power:GND #PWR057
 U 1 1 5C29DC0A
 P 3300 4200
-F 0 "#PWR07" H 3300 3950 50  0001 C CNN
+F 0 "#PWR057" H 3300 3950 50  0001 C CNN
 F 1 "GND" H 3300 4050 50  0000 C CNN
 F 2 "" H 3300 4200 50  0000 C CNN
@@
 	3300 4200 3300 3800
 $Comp
-L power:+BATT #PWR06
+L power:+BATT #PWR056
 U 1 1 5C29DEF5
 P 3300 3100
-F 0 "#PWR06" H 3300 2950 50  0001 C CNN
+F 0 "#PWR056" H 3300 2950 50  0001 C CNN
 F 1 "+BATT" H 3300 3240 50  0000 C CNN
 F 2 "" H 3300 3100 50  0000 C CNN

Commit message: KiCad: update pcb
Parts:
- C21, C22, C23: symbol Device:C -> KERISE-rescue:C-Device-KERISE-rescue-KERISE-rescue
- J14, J15: symbol Connector_Generic:Conn_01x02 -> KERISE-rescue:Conn_01x02-Connector_Generic-KERISE-rescue-KERISE-rescue
- L1, L2: symbol Device:L -> KERISE-rescue:L-Device-KERISE-rescue-KERISE-rescue
Changed lines of the file:
@@
 $EndComp
 $Comp
-L power:GND #PWR062
+L KERISE-rescue:GND-power-KERISE-rescue-KERISE-rescue #PWR061
 U 1 1 57CA1E46
 P 4800 4200
-F 0 "#PWR062" H 4800 3950 50  0001 C CNN
+F 0 "#PWR061" H 4800 3950 50  0001 C CNN
 F 1 "GND" H 4800 4050 50  0000 C CNN
 F 2 "" H 4800 4200 50  0000 C CNN
@@
 Motor
 $Comp
-L Device:C C23
+L KERISE-rescue:C-Device-KERISE-rescue-KERISE-rescue C23
 U 1 1 57CCEFE0
 P 4000 3650
@@
 $EndComp
 $Comp
-L power:+BATT #PWR065
+L KERISE-rescue:+BATT-power-KERISE-rescue-KERISE-rescue #PWR064
 U 1 1 57CD5BEE
 P 5600 3100
-F 0 "#PWR065" H 5600 2950 50  0001 C CNN
+F 0 "#PWR064" H 5600 2950 50  0001 C CNN
 F 1 "+BATT" H 5600 3240 50  0000 C CNN
 F 2 "" H 5600 3100 50  0000 C CNN
@@
 MT_OUT_R2
 $Comp
-L power:+3.3V #PWR063
+L KERISE-rescue:+3.3V-power-KERISE-rescue-KERISE-rescue #PWR?
 U 1 1 589CC6A5
 P 5300 3100
-F 0 "#PWR063" H 5300 2950 50  0001 C CNN
+AR Path="/589CC6A5" Ref="#PWR?"  Part="1"
+AR Path="/57CA18F6/589CC6A5" Ref="#PWR062"  Part="1"
+F 0 "#PWR062" H 5300 2950 50  0001 C CNN
 F 1 "+3.3V" H 5300 3240 50  0000 C CNN
 F 2 "" H 5300 3100 50  0000 C CNN
@@
 $EndComp
 $Comp
-L power:+3.3V #PWR060
+L KERISE-rescue:+3.3V-power-KERISE-rescue-KERISE-rescue #PWR?
 U 1 1 589CC6C6
 P 4000 3100
-F 0 "#PWR060" H 4000 2950 50  0001 C CNN
+AR Path="/589CC6C6" Ref="#PWR?"  Part="1"
+AR Path="/57CA18F6/589CC6C6" Ref="#PWR059"  Part="1"
+F 0 "#PWR059" H 4000 2950 50  0001 C CNN
 F 1 "+3.3V" H 4000 3240 50  0000 C CNN
 F 2 "" H 4000 3100 50  0000 C CNN
@@
 $EndComp
 $Comp
-L power:+BATT #PWR058
+L KERISE-rescue:+BATT-power-KERISE-rescue-KERISE-rescue #PWR057
 U 1 1 594721DF
 P 3700 3100
-F 0 "#PWR058" H 3700 2950 50  0001 C CNN
+F 0 "#PWR057" H 3700 2950 50  0001 C CNN
 F 1 "+BATT" H 3700 3240 50  0000 C CNN
 F 2 "" H 3700 3100 50  0000 C CNN
@@
 $EndComp
 $Comp
-L Device:C C22
+L KERISE-rescue:C-Device-KERISE-rescue-KERISE-rescue C22
 U 1 1 594721FA
 P 3700 3650
@@
 $EndComp
 $Comp
-L Device:L L1
+L KERISE-rescue:L-Device-KERISE-rescue-KERISE-rescue L1
 U 1 1 5B66FC72
 P 6350 3500
@@
 $EndComp
 $Comp
-L Device:L L2
+L KERISE-rescue:L-Device-KERISE-rescue-KERISE-rescue L2
 U 1 1 5B66FD2C
 P 6650 3600
@@
 MT_OUT_L_R
 $Comp
-L Connector_Generic:Conn_01x02 J14
+L KERISE-rescue:Conn_01x02-Connector_Generic-KERISE-rescue-KERISE-rescue J14
 U 1 1 5B6F504A
 P 8400 3400
@@
 $EndComp
 $Comp
-L Connector_Generic:Conn_01x02 J15
+L KERISE-rescue:Conn_01x02-Connector_Generic-KERISE-rescue-KERISE-rescue J15
 U 1 1 5B6F50A6
 P 8400 3900
@@
 $EndComp
 $Comp
-L power:GND #PWR066
+L KERISE-rescue:GND-power-KERISE-rescue-KERISE-rescue #PWR065
 U 1 1 5B6FD311
 P 5700 4200
-F 0 "#PWR066" H 5700 3950 50  0001 C CNN
+F 0 "#PWR065" H 5700 3950 50  0001 C CNN
 F 1 "GND" H 5700 4050 50  0000 C CNN
 F 2 "" H 5700 4200 50  0000 C CNN
@@
 $EndComp
 $Comp
-L power:GND #PWR061
+L KERISE-rescue:GND-power-KERISE-rescue-KERISE-rescue #PWR060
 U 1 1 5B6FD364
 P 4000 4200
-F 0 "#PWR061" H 4000 3950 50  0001 C CNN
+F 0 "#PWR060" H 4000 3950 50  0001 C CNN
 F 1 "GND" H 4000 4050 50  0000 C CNN
 F 2 "" H 4000 4200 50  0000 C CNN
@@
 $EndComp
 $Comp
-L power:GND #PWR059
+L KERISE-rescue:GND-power-KERISE-rescue-KERISE-rescue #PWR058
 U 1 1 5B7097B0
 P 3700 4200
-F 0 "#PWR059" H 3700 3950 50  0001 C CNN
+F 0 "#PWR058" H 3700 3950 50  0001 C CNN
 F 1 "GND" H 3700 4050 50  0000 C CNN
 F 2 "" H 3700 4200 50  0000 C CNN
@@
 $EndComp
 $Comp
-L power:GND #PWR064
+L KERISE-rescue:GND-power-KERISE-rescue-KERISE-rescue #PWR063
 U 1 1 5B7097C9
 P 5400 4200
-F 0 "#PWR064" H 5400 3950 50  0001 C CNN
+F 0 "#PWR063" H 5400 3950 50  0001 C CNN
 F 1 "GND" H 5400 4050 50  0000 C CNN
 F 2 "" H 5400 4200 50  0000 C CNN
@@
 $EndComp
 $Comp
-L Device:C C21
+L KERISE-rescue:C-Device-KERISE-rescue-KERISE-rescue C21
 U 1 1 5C29DB96
 P 3300 3650
@@
 $EndComp
 $Comp
-L power:GND #PWR057
+L KERISE-rescue:GND-power-KERISE-rescue-KERISE-rescue #PWR056
 U 1 1 5C29DC0A
 P 3300 4200
-F 0 "#PWR057" H 3300 3950 50  0001 C CNN
+F 0 "#PWR056" H 3300 3950 50  0001 C CNN
 F 1 "GND" H 3300 4050 50  0000 C CNN
 F 2 "" H 3300 4200 50  0000 C CNN
@@
 	3300 4200 3300 3800
 $Comp
-L power:+BATT #PWR056
+L KERISE-rescue:+BATT-power-KERISE-rescue-KERISE-rescue #PWR055
 U 1 1 5C29DEF5
 P 3300 3100
-F 0 "#PWR056" H 3300 2950 50  0001 C CNN
+F 0 "#PWR055" H 3300 2950 50  0001 C CNN
 F 1 "+BATT" H 3300 3240 50  0000 C CNN
 F 2 "" H 3300 3100 50  0000 C CNN
