File: kicad/Power.sch (KiCad schematic (older format))
At the start: 11 parts, among them U3 LXDC2UR30

Commit message: 予備配線完了
Parts:
- renumbered C5 to C18, C6 to C19, C7 to C20, D2 to D10, D1 to D9, R2 to R13, R3 to R14, R4 to R15, R5 to R16, U3 to U7
Changed lines of the file:
@@
 $Descr A4 11693 8268
 encoding utf-8
-Sheet 3 13
+Sheet 12 13
 Title ""
 Date ""
@@
 $EndDescr
 $Comp
-L power:+BATT #PWR017
+L power:+BATT #PWR038
 U 1 1 57CC111A
 P 2000 4200
-F 0 "#PWR017" H 2000 4050 50  0001 C CNN
+F 0 "#PWR038" H 2000 4050 50  0001 C CNN
 F 1 "+BATT" H 2000 4340 50  0000 C CNN
 F 2 "" H 2000 4200 50  0000 C CNN
@@
 Power
 $Comp
-L Device:R R2
+L Device:R R13
 U 1 1 57CD3B50
 P 3000 4450
-F 0 "R2" V 3080 4450 50  0000 C CNN
+F 0 "R13" V 3080 4450 50  0000 C CNN
 F 1 "10k" V 3000 4450 50  0000 C CNN
 F 2 "Resistor_SMD:R_0201_0603Metric" V 2930 4450 50  0001 C CNN
@@
 $EndComp
 $Comp
-L Device:R R3
+L Device:R R14
 U 1 1 57CD3B95
 P 3000 4950
-F 0 "R3" V 3080 4950 50  0000 C CNN
+F 0 "R14" V 3080 4950 50  0000 C CNN
 F 1 "10k" V 3000 4950 50  0000 C CNN
 F 2 "Resistor_SMD:R_0201_0603Metric" V 2930 4950 50  0001 C CNN
@@
 BAT_VOL
 $Comp
-L power:PWR_FLAG #FLG02
+L power:PWR_FLAG #FLG08
 U 1 1 57D18DE7
 P 2600 5100
-F 0 "#FLG02" H 2600 5195 50  0001 C CNN
+F 0 "#FLG08" H 2600 5195 50  0001 C CNN
 F 1 "PWR_FLAG" H 2600 5280 50  0000 C CNN
 F 2 "" H 2600 5100 50  0000 C CNN
@@
 $EndComp
 $Comp
-L power:PWR_FLAG #FLG01
+L power:PWR_FLAG #FLG07
 U 1 1 57D1915C
 P 2600 4300
-F 0 "#FLG01" H 2600 4395 50  0001 C CNN
+F 0 "#FLG07" H 2600 4395 50  0001 C CNN
 F 1 "PWR_FLAG" H 2600 4480 50  0000 C CNN
 F 2 "" H 2600 4300 50  0000 C CNN
@@
 $EndComp
 $Comp
-L power:+BATT #PWR019
+L power:+BATT #PWR040
 U 1 1 57D1923B
 P 2600 4200
-F 0 "#PWR019" H 2600 4050 50  0001 C CNN
+F 0 "#PWR040" H 2600 4050 50  0001 C CNN
 F 1 "+BATT" H 2600 4340 50  0000 C CNN
 F 2 "" H 2600 4200 50  0000 C CNN
@@
 $EndComp
 $Comp
-L Device:R R4
+L Device:R R15
 U 1 1 57D00960
 P 6600 4450
-F 0 "R4" V 6680 4450 50  0000 C CNN
+F 0 "R15" V 6680 4450 50  0000 C CNN
 F 1 "1k" V 6600 4450 50  0000 C CNN
 F 2 "Resistor_SMD:R_0201_0603Metric" V 6530 4450 50  0001 C CNN
@@
 $EndComp
 $Comp
-L power:GND #PWR032
+L power:GND #PWR053
 U 1 1 57D00A42
 P 6600 5200
-F 0 "#PWR032" H 6600 4950 50  0001 C CNN
+F 0 "#PWR053" H 6600 4950 50  0001 C CNN
 F 1 "GND" H 6600 5050 50  0000 C CNN
 F 2 "" H 6600 5200 50  0000 C CNN
@@
 $EndComp
 $Comp
-L power:+BATT #PWR021
+L power:+BATT #PWR042
 U 1 1 57CD3CA2
 P 3000 4200
-F 0 "#PWR021" H 3000 4050 50  0001 C CNN
+F 0 "#PWR042" H 3000 4050 50  0001 C CNN
 F 1 "+BATT" H 3000 4340 50  0000 C CNN
 F 2 "" H 3000 4200 50  0000 C CNN
@@
 $EndComp
 $Comp
-L power:+3.3V #PWR031
+L power:+3.3V #PWR052
 U 1 1 589CB64F
 P 6600 4200
-F 0 "#PWR031" H 6600 4050 50  0001 C CNN
+F 0 "#PWR052" H 6600 4050 50  0001 C CNN
 F 1 "+3.3V" H 6600 4340 50  0000 C CNN
 F 2 "" H 6600 4200 50  0000 C CNN
@@
 $EndComp
 $Comp
-L KERISE:LXDC2URxx U3
+L KERISE:LXDC2URxx U7
 U 1 1 592A4EE7
 P 5000 4250
-F 0 "U3" H 5000 4400 60  0000 C CNN
+F 0 "U7" H 5000 4400 60  0000 C CNN
 F 1 "LXDC2UR30" H 5000 4250 60  0000 C CNN
 F 2 "mouse:LXDC2UR" H 5000 4250 60  0001 C CNN
@@
 $EndComp
 $Comp
-L power:+BATT #PWR026
+L power:+BATT #PWR047
 U 1 1 592A5000
 P 4400 4200
-F 0 "#PWR026" H 4400 4050 50  0001 C CNN
+F 0 "#PWR047" H 4400 4050 50  0001 C CNN
 F 1 "+BATT" H 4400 4340 50  0000 C CNN
 F 2 "" H 4400 4200 50  0000 C CNN
@@
 Connection ~ 5600 4400
 $Comp
-L Device:LED D1
+L Device:LED D9
 U 1 1 594AB638
 P 6600 4850
-F 0 "D1" H 6600 4950 50  0000 C CNN
+F 0 "D9" H 6600 4950 50  0000 C CNN
 F 1 "Power" H 6600 4750 50  0000 C CNN
 F 2 "LED_SMD:LED_0402_1005Metric" H 6600 4850 50  0001 C CNN
@@
 	6600 5000 6600 5200
 $Comp
-L Device:C_Small C5
+L Device:C_Small C18
 U 1 1 59C47577
 P 3300 5000
-F 0 "C5" H 3310 5070 50  0000 L CNN
+F 0 "C18" H 3310 5070 50  0000 L CNN
 F 1 "0.1u" H 3310 4920 50  0000 L CNN
 F 2 "Capacitor_SMD:C_0201_0603Metric" H 3300 5000 50  0001 C CNN
@@
 	3300 5100 3300 5200
 $Comp
-L Device:R R5
+L Device:R R16
 U 1 1 5A4BB521
 P 6900 4450
-F 0 "R5" V 6980 4450 50  0000 C CNN
+F 0 "R16" V 6980 4450 50  0000 C CNN
 F 1 "1k" V 6900 4450 50  0000 C CNN
 F 2 "Resistor_SMD:R_0201_0603Metric" V 6830 4450 50  0001 C CNN
@@
 $EndComp
 $Comp
-L power:GND #PWR034
+L power:GND #PWR055
 U 1 1 5A4BB527
 P 6900 5200
-F 0 "#PWR034" H 6900 4950 50  0001 C CNN
+F 0 "#PWR055" H 6900 4950 50  0001 C CNN
 F 1 "GND" H 6900 5050 50  0000 C CNN
 F 2 "" H 6900 5200 50  0000 C CNN
@@
 $EndComp
 $Comp
-L power:+3.3V #PWR033
+L power:+3.3V #PWR054
 U 1 1 5A4BB52D
 P 6900 4200
-F 0 "#PWR033" H 6900 4050 50  0001 C CNN
+F 0 "#PWR054" H 6900 4050 50  0001 C CNN
 F 1 "+3.3V" H 6900 4340 50  0000 C CNN
 F 2 "" H 6900 4200 50  0000 C CNN
@@
 	6900 4300 6900 4200
 $Comp
-L Device:LED D2
+L Device:LED D10
 U 1 1 5A4BB535
 P 6900 4850
-F 0 "D2" H 6900 4950 50  0000 C CNN
+F 0 "D10" H 6900 4950 50  0000 C CNN
 F 1 "Power" H 6900 4750 50  0000 C CNN
 F 2 "LED_SMD:LED_0402_1005Metric" H 6900 4850 50  0001 C CNN
@@
 	3000 4700 3000 4800
 $Comp
-L power:GND #PWR022
+L power:GND #PWR043
 U 1 1 5B6FEDB1
 P 3000 5200
-F 0 "#PWR022" H 3000 4950 50  0001 C CNN
+F 0 "#PWR043" H 3000 4950 50  0001 C CNN
 F 1 "GND" H 3000 5050 50  0000 C CNN
 F 2 "" H 3000 5200 50  0000 C CNN
@@
 $EndComp
 $Comp
-L power:GND #PWR023
+L power:GND #PWR044
 U 1 1 5B6FEDD6
 P 3300 5200
-F 0 "#PWR023" H 3300 4950 50  0001 C CNN
+F 0 "#PWR044" H 3300 4950 50  0001 C CNN
 F 1 "GND" H 3300 5050 50  0000 C CNN
 F 2 "" H 3300 5200 50  0000 C CNN
@@
 $EndComp
 $Comp
-L power:GND #PWR020
+L power:GND #PWR041
 U 1 1 5B705567
 P 2600 5200
-F 0 "#PWR020" H 2600 4950 50  0001 C CNN
+F 0 "#PWR041" H 2600 4950 50  0001 C CNN
 F 1 "GND" H 2600 5050 50  0000 C CNN
 F 2 "" H 2600 5200 50  0000 C CNN
@@
 $EndComp
 $Comp
-L power:GND #PWR027
+L power:GND #PWR048
 U 1 1 5B70558C
 P 5000 5200
-F 0 "#PWR027" H 5000 4950 50  0001 C CNN
+F 0 "#PWR048" H 5000 4950 50  0001 C CNN
 F 1 "GND" H 5000 5050 50  0000 C CNN
 F 2 "" H 5000 5200 50  0000 C CNN
@@
 $EndComp
 $Comp
-L power:+3.3V #PWR028
+L power:+3.3V #PWR049
 U 1 1 5B705DFE
 P 5600 4200
-F 0 "#PWR028" H 5600 4050 50  0001 C CNN
+F 0 "#PWR049" H 5600 4050 50  0001 C CNN
 F 1 "+3.3V" H 5600 4340 50  0000 C CNN
 F 2 "" H 5600 4200 50  0000 C CNN
@@
 $EndComp
 $Comp
-L power:GND #PWR018
+L power:GND #PWR039
 U 1 1 5B707C07
 P 2000 5200
-F 0 "#PWR018" H 2000 4950 50  0001 C CNN
+F 0 "#PWR039" H 2000 4950 50  0001 C CNN
 F 1 "GND" H 2000 5050 50  0000 C CNN
 F 2 "" H 2000 5200 50  0000 C CNN
@@
 $EndComp
 $Comp
-L Device:C C7
+L Device:C C20
 U 1 1 5B93EBC5
 P 5900 4750
-F 0 "C7" H 6015 4796 50  0000 L CNN
+F 0 "C20" H 6015 4796 50  0000 L CNN
 F 1 "47u" H 6015 4705 50  0000 L CNN
 F 2 "Capacitor_SMD:C_0805_2012Metric" H 5938 4600 50  0001 C CNN
@@
 $EndComp
 $Comp
-L power:GND #PWR030
+L power:GND #PWR051
 U 1 1 5B93EC2F
 P 5900 5200
-F 0 "#PWR030" H 5900 4950 50  0001 C CNN
+F 0 "#PWR051" H 5900 4950 50  0001 C CNN
 F 1 "GND" H 5900 5050 50  0000 C CNN
 F 2 "" H 5900 5200 50  0000 C CNN
@@
 	5900 4900 5900 5200
 $Comp
-L power:+3.3V #PWR029
+L power:+3.3V #PWR050
 U 1 1 5B93F57B
 P 5900 4200
-F 0 "#PWR029" H 5900 4050 50  0001 C CNN
+F 0 "#PWR050" H 5900 4050 50  0001 C CNN
 F 1 "+3.3V" H 5900 4340 50  0000 C CNN
 F 2 "" H 5900 4200 50  0000 C CNN
@@
 	5900 4200 5900 4600
 $Comp
-L Device:C C6
+L Device:C C19
 U 1 1 5C2A0D61
 P 4100 4750
-F 0 "C6" H 4215 4796 50  0000 L CNN
+F 0 "C19" H 4215 4796 50  0000 L CNN
 F 1 "47u" H 4215 4705 50  0000 L CNN
 F 2 "Capacitor_SMD:C_0805_2012Metric" H 4138 4600 50  0001 C CNN
@@
 $EndComp
 $Comp
-L power:+BATT #PWR024
+L power:+BATT #PWR045
 U 1 1 5C2A0DD3
 P 4100 4200
-F 0 "#PWR024" H 4100 4050 50  0001 C CNN
+F 0 "#PWR045" H 4100 4050 50  0001 C CNN
 F 1 "+BATT" H 4100 4340 50  0000 C CNN
 F 2 "" H 4100 4200 50  0000 C CNN
@@
 $EndComp
 $Comp
-L power:GND #PWR025
+L power:GND #PWR046
 U 1 1 5C2A0DF8
 P 4100 5200
-F 0 "#PWR025" H 4100 4950 50  0001 C CNN
+F 0 "#PWR046" H 4100 4950 50  0001 C CNN
 F 1 "GND" H 4100 5050 50  0000 C CNN
 F 2 "" H 4100 5200 50  0000 C CNN

Commit message: KiCad: update pcb
Parts:
- BT1: symbol Device:Battery_Cell -> KERISE-rescue:Battery_Cell-Device-KERISE-rescue-KERISE-rescue
- C18: symbol Device:C_Small -> KERISE-rescue:C_Small-Device-KERISE-rescue-KERISE-rescue
- C19, C20: symbol Device:C -> KERISE-rescue:C-Device-KERISE-rescue-KERISE-rescue
- D10, D9: symbol Device:LED -> KERISE-rescue:LED-Device-KERISE-rescue-KERISE-rescue
- R13, R14, R15, R16: symbol Device:R -> KERISE-rescue:R-Device-KERISE-rescue-KERISE-rescue
Changed lines of the file:
@@
 $EndDescr
 $Comp
-L power:+BATT #PWR038
+L KERISE-rescue:+BATT-power-KERISE-rescue-KERISE-rescue #PWR037
 U 1 1 57CC111A
 P 2000 4200
-F 0 "#PWR038" H 2000 4050 50  0001 C CNN
+F 0 "#PWR037" H 2000 4050 50  0001 C CNN
 F 1 "+BATT" H 2000 4340 50  0000 C CNN
 F 2 "" H 2000 4200 50  0000 C CNN
@@
 Power
 $Comp
-L Device:R R13
+L KERISE-rescue:R-Device-KERISE-rescue-KERISE-rescue R13
 U 1 1 57CD3B50
 P 3000 4450
@@
 $EndComp
 $Comp
-L Device:R R14
+L KERISE-rescue:R-Device-KERISE-rescue-KERISE-rescue R14
 U 1 1 57CD3B95
 P 3000 4950
@@
 BAT_VOL
 $Comp
-L power:PWR_FLAG #FLG08
+L KERISE-rescue:PWR_FLAG-power-KERISE-rescue-KERISE-rescue #FLG08
 U 1 1 57D18DE7
 P 2600 5100
@@
 $EndComp
 $Comp
-L power:PWR_FLAG #FLG07
+L KERISE-rescue:PWR_FLAG-power-KERISE-rescue-KERISE-rescue #FLG07
 U 1 1 57D1915C
 P 2600 4300
@@
 $EndComp
 $Comp
-L power:+BATT #PWR040
+L KERISE-rescue:+BATT-power-KERISE-rescue-KERISE-rescue #PWR039
 U 1 1 57D1923B
 P 2600 4200
-F 0 "#PWR040" H 2600 4050 50  0001 C CNN
+F 0 "#PWR039" H 2600 4050 50  0001 C CNN
 F 1 "+BATT" H 2600 4340 50  0000 C CNN
 F 2 "" H 2600 4200 50  0000 C CNN
@@
 $EndComp
 $Comp
-L Device:R R15
+L KERISE-rescue:R-Device-KERISE-rescue-KERISE-rescue R15
 U 1 1 57D00960
 P 6600 4450
@@
 $EndComp
 $Comp
-L power:GND #PWR053
+L KERISE-rescue:GND-power-KERISE-rescue-KERISE-rescue #PWR052
 U 1 1 57D00A42
 P 6600 5200
-F 0 "#PWR053" H 6600 4950 50  0001 C CNN
+F 0 "#PWR052" H 6600 4950 50  0001 C CNN
 F 1 "GND" H 6600 5050 50  0000 C CNN
 F 2 "" H 6600 5200 50  0000 C CNN
@@
 $EndComp
 $Comp
-L power:+BATT #PWR042
+L KERISE-rescue:+BATT-power-KERISE-rescue-KERISE-rescue #PWR041
 U 1 1 57CD3CA2
 P 3000 4200
-F 0 "#PWR042" H 3000 4050 50  0001 C CNN
+F 0 "#PWR041" H 3000 4050 50  0001 C CNN
 F 1 "+BATT" H 3000 4340 50  0000 C CNN
 F 2 "" H 3000 4200 50  0000 C CNN
@@
 $EndComp
 $Comp
-L power:+3.3V #PWR052
+L KERISE-rescue:+3.3V-power-KERISE-rescue-KERISE-rescue #PWR?
 U 1 1 589CB64F
 P 6600 4200
-F 0 "#PWR052" H 6600 4050 50  0001 C CNN
+AR Path="/589CB64F" Ref="#PWR?"  Part="1"
+AR Path="/57CA15C1/589CB64F" Ref="#PWR051"  Part="1"
+F 0 "#PWR051" H 6600 4050 50  0001 C CNN
 F 1 "+3.3V" H 6600 4340 50  0000 C CNN
 F 2 "" H 6600 4200 50  0000 C CNN
@@
 $EndComp
 $Comp
-L power:+BATT #PWR047
+L KERISE-rescue:+BATT-power-KERISE-rescue-KERISE-rescue #PWR046
 U 1 1 592A5000
 P 4400 4200
-F 0 "#PWR047" H 4400 4050 50  0001 C CNN
+F 0 "#PWR046" H 4400 4050 50  0001 C CNN
 F 1 "+BATT" H 4400 4340 50  0000 C CNN
 F 2 "" H 4400 4200 50  0000 C CNN
@@
 Connection ~ 5600 4400
 $Comp
-L Device:LED D9
+L KERISE-rescue:LED-Device-KERISE-rescue-KERISE-rescue D9
 U 1 1 594AB638
 P 6600 4850
@@
 	6600 5000 6600 5200
 $Comp
-L Device:C_Small C18
+L KERISE-rescue:C_Small-Device-KERISE-rescue-KERISE-rescue C18
 U 1 1 59C47577
 P 3300 5000
@@
 	3300 5100 3300 5200
 $Comp
-L Device:R R16
+L KERISE-rescue:R-Device-KERISE-rescue-KERISE-rescue R16
 U 1 1 5A4BB521
 P 6900 4450
@@
 $EndComp
 $Comp
-L power:GND #PWR055
+L KERISE-rescue:GND-power-KERISE-rescue-KERISE-rescue #PWR054
 U 1 1 5A4BB527
 P 6900 5200
-F 0 "#PWR055" H 6900 4950 50  0001 C CNN
+F 0 "#PWR054" H 6900 4950 50  0001 C CNN
 F 1 "GND" H 6900 5050 50  0000 C CNN
 F 2 "" H 6900 5200 50  0000 C CNN
@@
 $EndComp
 $Comp
-L power:+3.3V #PWR054
+L KERISE-rescue:+3.3V-power-KERISE-rescue-KERISE-rescue #PWR?
 U 1 1 5A4BB52D
 P 6900 4200
-F 0 "#PWR054" H 6900 4050 50  0001 C CNN
+AR Path="/5A4BB52D" Ref="#PWR?"  Part="1"
+AR Path="/57CA15C1/5A4BB52D" Ref="#PWR053"  Part="1"
+F 0 "#PWR053" H 6900 4050 50  0001 C CNN
 F 1 "+3.3V" H 6900 4340 50  0000 C CNN
 F 2 "" H 6900 4200 50  0000 C CNN
@@
 	6900 4300 6900 4200
 $Comp
-L Device:LED D10
+L KERISE-rescue:LED-Device-KERISE-rescue-KERISE-rescue D10
 U 1 1 5A4BB535
 P 6900 4850
@@
 	3300 4700 3400 4700
 $Comp
-L Device:Battery_Cell BT1
+L KERISE-rescue:Battery_Cell-Device-KERISE-rescue-KERISE-rescue BT1
 U 1 1 5B6F55D7
 P 2000 4700
@@
 	3000 4700 3000 4800
 $Comp
-L power:GND #PWR043
+L KERISE-rescue:GND-power-KERISE-rescue-KERISE-rescue #PWR042
 U 1 1 5B6FEDB1
 P 3000 5200
-F 0 "#PWR043" H 3000 4950 50  0001 C CNN
+F 0 "#PWR042" H 3000 4950 50  0001 C CNN
 F 1 "GND" H 3000 5050 50  0000 C CNN
 F 2 "" H 3000 5200 50  0000 C CNN
@@
 $EndComp
 $Comp
-L power:GND #PWR044
+L KERISE-rescue:GND-power-KERISE-rescue-KERISE-rescue #PWR043
 U 1 1 5B6FEDD6
 P 3300 5200
-F 0 "#PWR044" H 3300 4950 50  0001 C CNN
+F 0 "#PWR043" H 3300 4950 50  0001 C CNN
 F 1 "GND" H 3300 5050 50  0000 C CNN
 F 2 "" H 3300 5200 50  0000 C CNN
@@
 $EndComp
 $Comp
-L power:GND #PWR041
+L KERISE-rescue:GND-power-KERISE-rescue-KERISE-rescue #PWR040
 U 1 1 5B705567
 P 2600 5200
-F 0 "#PWR041" H 2600 4950 50  0001 C CNN
+F 0 "#PWR040" H 2600 4950 50  0001 C CNN
 F 1 "GND" H 2600 5050 50  0000 C CNN
 F 2 "" H 2600 5200 50  0000 C CNN
@@
 $EndComp
 $Comp
-L power:GND #PWR048
+L KERISE-rescue:GND-power-KERISE-rescue-KERISE-rescue #PWR047
 U 1 1 5B70558C
 P 5000 5200
-F 0 "#PWR048" H 5000 4950 50  0001 C CNN
+F 0 "#PWR047" H 5000 4950 50  0001 C CNN
 F 1 "GND" H 5000 5050 50  0000 C CNN
 F 2 "" H 5000 5200 50  0000 C CNN
@@
 $EndComp
 $Comp
-L power:+3.3V #PWR049
+L KERISE-rescue:+3.3V-power-KERISE-rescue-KERISE-rescue #PWR?
 U 1 1 5B705DFE
 P 5600 4200
-F 0 "#PWR049" H 5600 4050 50  0001 C CNN
+AR Path="/5B705DFE" Ref="#PWR?"  Part="1"
+AR Path="/57CA15C1/5B705DFE" Ref="#PWR048"  Part="1"
+F 0 "#PWR048" H 5600 4050 50  0001 C CNN
 F 1 "+3.3V" H 5600 4340 50  0000 C CNN
 F 2 "" H 5600 4200 50  0000 C CNN
@@
 $EndComp
 $Comp
-L power:GND #PWR039
+L KERISE-rescue:GND-power-KERISE-rescue-KERISE-rescue #PWR038
 U 1 1 5B707C07
 P 2000 5200
-F 0 "#PWR039" H 2000 4950 50  0001 C CNN
+F 0 "#PWR038" H 2000 4950 50  0001 C CNN
 F 1 "GND" H 2000 5050 50  0000 C CNN
 F 2 "" H 2000 5200 50  0000 C CNN
@@
 $EndComp
 $Comp
-L Device:C C20
+L KERISE-rescue:C-Device-KERISE-rescue-KERISE-rescue C20
 U 1 1 5B93EBC5
 P 5900 4750
@@
 $EndComp
 $Comp
-L power:GND #PWR051
+L KERISE-rescue:GND-power-KERISE-rescue-KERISE-rescue #PWR050
 U 1 1 5B93EC2F
 P 5900 5200
-F 0 "#PWR051" H 5900 4950 50  0001 C CNN
+F 0 "#PWR050" H 5900 4950 50  0001 C CNN
 F 1 "GND" H 5900 5050 50  0000 C CNN
 F 2 "" H 5900 5200 50  0000 C CNN
@@
 	5900 4900 5900 5200
 $Comp
-L power:+3.3V #PWR050
+L KERISE-rescue:+3.3V-power-KERISE-rescue-KERISE-rescue #PWR?
 U 1 1 5B93F57B
 P 5900 4200
-F 0 "#PWR050" H 5900 4050 50  0001 C CNN
+AR Path="/5B93F57B" Ref="#PWR?"  Part="1"
+AR Path="/57CA15C1/5B93F57B" Ref="#PWR049"  Part="1"
+F 0 "#PWR049" H 5900 4050 50  0001 C CNN
 F 1 "+3.3V" H 5900 4340 50  0000 C CNN
 F 2 "" H 5900 4200 50  0000 C CNN
@@
 	5900 4200 5900 4600
 $Comp
-L Device:C C19
+L KERISE-rescue:C-Device-KERISE-rescue-KERISE-rescue C19
 U 1 1 5C2A0D61
 P 4100 4750
@@
 $EndComp
 $Comp
-L power:+BATT #PWR045
+L KERISE-rescue:+BATT-power-KERISE-rescue-KERISE-rescue #PWR044
 U 1 1 5C2A0DD3
 P 4100 4200
-F 0 "#PWR045" H 4100 4050 50  0001 C CNN
+F 0 "#PWR044" H 4100 4050 50  0001 C CNN
 F 1 "+BATT" H 4100 4340 50  0000 C CNN
 F 2 "" H 4100 4200 50  0000 C CNN
@@
 $EndComp
 $Comp
-L power:GND #PWR046
+L KERISE-rescue:GND-power-KERISE-rescue-KERISE-rescue #PWR045
 U 1 1 5C2A0DF8
 P 4100 5200
-F 0 "#PWR046" H 4100 4950 50  0001 C CNN
+F 0 "#PWR045" H 4100 4950 50  0001 C CNN
 F 1 "GND" H 4100 5050 50  0000 C CNN
 F 2 "" H 4100 5200 50  0000 C CNN
