File: kicad/ToF.sch (KiCad schematic (older format))
At the start: 7 parts, among them P1 ToF_Host, P2 ToF_Slave, U8 VL6180X

Commit message: 予備配線完了
Parts:
- renumbered C22 to C2, C23 to C3, R15 to R2, R16 to R3, U8 to U2
Changed lines of the file:
@@
 SCL
 $Comp
-L Device:C_Small C23
+L Device:C_Small C3
 U 1 1 592BA26F
 P 3900 3800
-F 0 "C23" H 3910 3870 50  0000 L CNN
+F 0 "C3" H 3910 3870 50  0000 L CNN
 F 1 "0.1u" H 3910 3720 50  0000 L CNN
 F 2 "Capacitor_SMD:C_0201_0603Metric" H 3900 3800 50  0001 C CNN
@@
 $EndComp
 $Comp
-L Device:C_Small C22
+L Device:C_Small C2
 U 1 1 592BA2BF
 P 3600 3800
-F 0 "C22" H 3610 3870 50  0000 L CNN
+F 0 "C2" H 3610 3870 50  0000 L CNN
 F 1 "4.7u" H 3610 3720 50  0000 L CNN
 F 2 "Capacitor_SMD:C_0402_1005Metric" H 3600 3800 50  0001 C CNN
@@
 	5400 3400 5300 3400
 $Comp
-L Device:R R15
+L Device:R R2
 U 1 1 5AB6394F
 P 5700 3450
-F 0 "R15" V 5780 3450 50  0000 C CNN
+F 0 "R2" V 5780 3450 50  0000 C CNN
 F 1 "4.7k" V 5700 3450 50  0000 C CNN
 F 2 "Resistor_SMD:R_0201_0603Metric" V 5630 3450 50  0001 C CNN
@@
 $EndComp
 $Comp
-L Device:R R16
+L Device:R R3
 U 1 1 5AB639A9
 P 5900 3450
-F 0 "R16" V 5980 3450 50  0000 C CNN
+F 0 "R3" V 5980 3450 50  0000 C CNN
 F 1 "4.7k" V 5900 3450 50  0000 C CNN
 F 2 "Resistor_SMD:R_0201_0603Metric" V 5830 3450 50  0001 C CNN
@@
 	4200 3400 4200 3500
 $Comp
-L power:GND #PWR066
+L power:GND #PWR07
 U 1 1 5C29A844
 P 4300 2700
-F 0 "#PWR066" H 4300 2450 50  0001 C CNN
+F 0 "#PWR07" H 4300 2450 50  0001 C CNN
 F 1 "GND" H 4305 2527 50  0000 C CNN
 F 2 "" H 4300 2700 50  0001 C CNN
@@
 $EndComp
 $Comp
-L power:+3.3V #PWR065
+L power:+3.3V #PWR06
 U 1 1 5C29A8B4
 P 4300 2200
-F 0 "#PWR065" H 4300 2050 50  0001 C CNN
+F 0 "#PWR06" H 4300 2050 50  0001 C CNN
 F 1 "+3.3V" H 4315 2373 50  0000 C CNN
 F 2 "" H 4300 2200 50  0001 C CNN
@@
 $EndComp
 $Comp
-L power:PWR_FLAG #FLG07
+L power:PWR_FLAG #FLG01
 U 1 1 5C29AA5D
 P 5300 2300
-F 0 "#FLG07" H 5300 2375 50  0001 C CNN
+F 0 "#FLG01" H 5300 2375 50  0001 C CNN
 F 1 "PWR_FLAG" H 5300 2474 50  0000 C CNN
 F 2 "" H 5300 2300 50  0001 C CNN
@@
 $EndComp
 $Comp
-L power:PWR_FLAG #FLG08
+L power:PWR_FLAG #FLG02
 U 1 1 5C29B1AD
 P 5300 2600
-F 0 "#FLG08" H 5300 2675 50  0001 C CNN
+F 0 "#FLG02" H 5300 2675 50  0001 C CNN
 F 1 "PWR_FLAG" H 5300 2773 50  0000 C CNN
 F 2 "" H 5300 2600 50  0001 C CNN
@@
 $EndComp
 $Comp
-L KERISE:VL6180X U8
+L KERISE:VL6180X U2
 U 1 1 5C29B6B0
 P 4800 3300
-F 0 "U8" H 4800 3587 60  0000 C CNN
+F 0 "U2" H 4800 3587 60  0000 C CNN
 F 1 "VL6180X" H 4800 3481 60  0000 C CNN
 F 2 "mouse:VL6180X" H 4800 3300 60  0001 C CNN

Commit message: KiCad: update pcb
Parts:
- C2, C3: symbol Device:C_Small -> KERISE-rescue:C_Small-Device-KERISE-rescue-KERISE-rescue
- P1: symbol Connector:Conn_01x04_Female -> KERISE-rescue:Conn_01x04_Female-Connector-KERISE-rescue-KERISE-rescue
- P2: symbol Connector:Conn_01x04_Male -> KERISE-rescue:Conn_01x04_Male-Connector-KERISE-rescue-KERISE-rescue
- R2, R3: symbol Device:R -> KERISE-rescue:R-Device-KERISE-rescue-KERISE-rescue
Changed lines of the file:
@@
 SCL
 $Comp
-L Device:C_Small C3
+L KERISE-rescue:C_Small-Device-KERISE-rescue-KERISE-rescue C3
 U 1 1 592BA26F
 P 3900 3800
@@
 $EndComp
 $Comp
-L Device:C_Small C2
+L KERISE-rescue:C_Small-Device-KERISE-rescue-KERISE-rescue C2
 U 1 1 592BA2BF
 P 3600 3800
@@
 s_GND
 $Comp
-L Connector:Conn_01x04_Male P2
+L KERISE-rescue:Conn_01x04_Male-Connector-KERISE-rescue-KERISE-rescue P2
 U 1 1 592AB803
 P 5000 2400
@@
 	5400 3400 5300 3400
 $Comp
-L Device:R R2
+L KERISE-rescue:R-Device-KERISE-rescue-KERISE-rescue R2
 U 1 1 5AB6394F
 P 5700 3450
@@
 $EndComp
 $Comp
-L Device:R R3
+L KERISE-rescue:R-Device-KERISE-rescue-KERISE-rescue R3
 U 1 1 5AB639A9
 P 5900 3450
@@
 	4200 3400 4200 3500
 $Comp
-L power:GND #PWR07
+L KERISE-rescue:GND-power-KERISE-rescue-KERISE-rescue #PWR07
 U 1 1 5C29A844
 P 4300 2700
@@
 $EndComp
 $Comp
-L power:+3.3V #PWR06
+L KERISE-rescue:+3.3V-power-KERISE-rescue-KERISE-rescue #PWR?
 U 1 1 5C29A8B4
 P 4300 2200
+AR Path="/5C29A8B4" Ref="#PWR?"  Part="1"
+AR Path="/5C29A0B1/5C29A8B4" Ref="#PWR06"  Part="1"
 F 0 "#PWR06" H 4300 2050 50  0001 C CNN
 F 1 "+3.3V" H 4315 2373 50  0000 C CNN
@@
 $EndComp
 $Comp
-L Connector:Conn_01x04_Female P1
+L KERISE-rescue:Conn_01x04_Female-Connector-KERISE-rescue-KERISE-rescue P1
 U 1 1 592AB778
 P 4600 2400
@@
 $EndComp
 $Comp
-L power:PWR_FLAG #FLG01
+L KERISE-rescue:PWR_FLAG-power-KERISE-rescue-KERISE-rescue #FLG01
 U 1 1 5C29AA5D
 P 5300 2300
@@
 $EndComp
 $Comp
-L power:PWR_FLAG #FLG02
+L KERISE-rescue:PWR_FLAG-power-KERISE-rescue-KERISE-rescue #FLG02
 U 1 1 5C29B1AD
 P 5300 2600
