File: kicad/UI.sch (KiCad schematic (older format))
At the start: 12 parts, among them Q13 DMN3065LW-7, SW2 UPLOAD, U7 PCA9632

Commit message: 予備配線完了
Parts:
- renumbered C20 to C4, C21 to C5, D7 to D1, D8 to D2, D9 to D3, D10 to D4, Q13 to Q1, R14 to R4, U7 to U3
Changed lines of the file:
@@
 $EndDescr
 $Comp
-L power:GND #PWR060
+L power:GND #PWR015
 U 1 1 57CEA2EF
 P 6500 4600
-F 0 "#PWR060" H 6500 4350 50  0001 C CNN
+F 0 "#PWR015" H 6500 4350 50  0001 C CNN
 F 1 "GND" H 6500 4450 50  0000 C CNN
 F 2 "" H 6500 4600 50  0000 C CNN
@@
 	6500 4600 6500 4400
 $Comp
-L power:GND #PWR062
+L power:GND #PWR017
 U 1 1 5A1C53C4
 P 7900 4600
-F 0 "#PWR062" H 7900 4350 50  0001 C CNN
+F 0 "#PWR017" H 7900 4350 50  0001 C CNN
 F 1 "GND" H 7900 4450 50  0000 C CNN
 F 2 "" H 7900 4600 50  0000 C CNN
@@
 SDA
 $Comp
-L power:+3.3V #PWR054
+L power:+3.3V #PWR09
 U 1 1 5A202D5A
 P 4050 2950
-F 0 "#PWR054" H 4050 2800 50  0001 C CNN
+F 0 "#PWR09" H 4050 2800 50  0001 C CNN
 F 1 "+3.3V" H 4050 3090 50  0000 C CNN
 F 2 "" H 4050 2950 50  0001 C CNN
@@
 	4050 2950 4050 3050
 $Comp
-L power:GND #PWR055
+L power:GND #PWR010
 U 1 1 5A202F53
 P 4050 4650
-F 0 "#PWR055" H 4050 4400 50  0001 C CNN
+F 0 "#PWR010" H 4050 4400 50  0001 C CNN
 F 1 "GND" H 4050 4500 50  0000 C CNN
 F 2 "" H 4050 4650 50  0000 C CNN
@@
 	5050 3050 5050 2950
 $Comp
-L power:+3.3V #PWR057
+L power:+3.3V #PWR012
 U 1 1 5A204571
 P 5050 2950
-F 0 "#PWR057" H 5050 2800 50  0001 C CNN
+F 0 "#PWR012" H 5050 2800 50  0001 C CNN
 F 1 "+3.3V" H 5050 3090 50  0000 C CNN
 F 2 "" H 5050 2950 50  0001 C CNN
@@
 $EndComp
 $Comp
-L Device:LED_Small D8
+L Device:LED_Small D2
 U 1 1 5A204565
 P 5050 3150
-F 0 "D8" H 5000 3275 50  0000 L CNN
+F 0 "D2" H 5000 3275 50  0000 L CNN
 F 1 "LED" H 5000 3050 50  0000 L CNN
 F 2 "LED_SMD:LED_0402_1005Metric" V 5050 3150 50  0001 C CNN
@@
 	4750 3050 4750 2950
 $Comp
-L power:+3.3V #PWR056
+L power:+3.3V #PWR011
 U 1 1 5A203D72
 P 4750 2950
-F 0 "#PWR056" H 4750 2800 50  0001 C CNN
+F 0 "#PWR011" H 4750 2800 50  0001 C CNN
 F 1 "+3.3V" H 4750 3090 50  0000 C CNN
 F 2 "" H 4750 2950 50  0001 C CNN
@@
 $EndComp
 $Comp
-L Device:LED_Small D7
+L Device:LED_Small D1
 U 1 1 5A203147
 P 4750 3150
-F 0 "D7" H 4700 3275 50  0000 L CNN
+F 0 "D1" H 4700 3275 50  0000 L CNN
 F 1 "LED" H 4700 3050 50  0000 L CNN
 F 2 "LED_SMD:LED_0402_1005Metric" V 4750 3150 50  0001 C CNN
@@
 	5650 3050 5650 2950
 $Comp
-L power:+3.3V #PWR059
+L power:+3.3V #PWR014
 U 1 1 5A20460C
 P 5650 2950
-F 0 "#PWR059" H 5650 2800 50  0001 C CNN
+F 0 "#PWR014" H 5650 2800 50  0001 C CNN
 F 1 "+3.3V" H 5650 3090 50  0000 C CNN
 F 2 "" H 5650 2950 50  0001 C CNN
@@
 $EndComp
 $Comp
-L Device:LED_Small D10
+L Device:LED_Small D4
 U 1 1 5A204618
 P 5650 3150
-F 0 "D10" H 5600 3275 50  0000 L CNN
+F 0 "D4" H 5600 3275 50  0000 L CNN
 F 1 "LED" H 5600 3050 50  0000 L CNN
 F 2 "LED_SMD:LED_0402_1005Metric" V 5650 3150 50  0001 C CNN
@@
 	5350 3050 5350 2950
 $Comp
-L power:+3.3V #PWR058
+L power:+3.3V #PWR013
 U 1 1 5A204620
 P 5350 2950
-F 0 "#PWR058" H 5350 2800 50  0001 C CNN
+F 0 "#PWR013" H 5350 2800 50  0001 C CNN
 F 1 "+3.3V" H 5350 3090 50  0000 C CNN
 F 2 "" H 5350 2950 50  0001 C CNN
@@
 $EndComp
 $Comp
-L Device:LED_Small D9
+L Device:LED_Small D3
 U 1 1 5A20462C
 P 5350 3150
-F 0 "D9" H 5300 3275 50  0000 L CNN
+F 0 "D3" H 5300 3275 50  0000 L CNN
 F 1 "LED" H 5300 3050 50  0000 L CNN
 F 2 "LED_SMD:LED_0402_1005Metric" V 5350 3150 50  0001 C CNN
@@
 $EndComp
 $Comp
-L Device:C_Small C20
+L Device:C_Small C4
 U 1 1 5A2A1F42
 P 3850 3250
-F 0 "C20" H 3860 3320 50  0000 L CNN
+F 0 "C4" H 3860 3320 50  0000 L CNN
 F 1 "0.1u" H 3860 3170 50  0000 L CNN
 F 2 "Capacitor_SMD:C_0201_0603Metric" H 3850 3250 50  0001 C CNN
@@
 $EndComp
 $Comp
-L power:GND #PWR053
+L power:GND #PWR08
 U 1 1 5A2A2041
 P 3850 3350
-F 0 "#PWR053" H 3850 3100 50  0001 C CNN
+F 0 "#PWR08" H 3850 3100 50  0001 C CNN
 F 1 "GND" H 3850 3200 50  0000 C CNN
 F 2 "" H 3850 3350 50  0001 C CNN
@@
 Connection ~ 4050 3050
 $Comp
-L KERISE:PCA9632 U7
+L KERISE:PCA9632 U3
 U 1 1 5A2BFCCE
 P 4050 4100
-F 0 "U7" H 3550 4425 50  0000 L CNN
+F 0 "U3" H 3550 4425 50  0000 L CNN
 F 1 "PCA9632" H 4100 4425 50  0000 L CNN
 F 2 "mouse:DFN-8-1EP_3x3mm_Pitch0.5mm" H 4100 3800 50  0001 L CNN
@@
 $EndComp
 $Comp
-L Device:Q_NMOS_GSD Q13
+L Device:Q_NMOS_GSD Q1
 U 1 1 5B6723D7
 P 7800 4300
-F 0 "Q13" H 7800 4450 50  0000 R CNN
+F 0 "Q1" H 7800 4450 50  0000 R CNN
 F 1 "DMN3065LW-7" H 7850 4150 50  0000 R CNN
 F 2 "Package_TO_SOT_SMD:SOT-323_SC-70" H 8000 4400 50  0001 C CNN
@@
 	7500 4300 7600 4300
 $Comp
-L Device:R R14
+L Device:R R4
 U 1 1 5B6725CD
 P 7900 3850
-F 0 "R14" V 7980 3850 50  0000 C CNN
+F 0 "R4" V 7980 3850 50  0000 C CNN
 F 1 "10" V 7900 3850 50  0000 C CNN
 F 2 "Resistor_SMD:R_0201_0603Metric" V 7830 3850 50  0001 C CNN
@@
 $EndComp
 $Comp
-L power:+BATT #PWR061
+L power:+BATT #PWR016
 U 1 1 5C29DB6A
 P 7900 3400
-F 0 "#PWR061" H 7900 3250 50  0001 C CNN
+F 0 "#PWR016" H 7900 3250 50  0001 C CNN
 F 1 "+BATT" H 7915 3573 50  0000 C CNN
 F 2 "" H 7900 3400 50  0001 C CNN
@@
 $EndComp
 $Comp
-L Device:C C21
+L Device:C C5
 U 1 1 5C29E0A6
 P 8600 4050
-F 0 "C21" H 8715 4096 50  0000 L CNN
+F 0 "C5" H 8715 4096 50  0000 L CNN
 F 1 "10u" H 8715 4005 50  0000 L CNN
 F 2 "Capacitor_SMD:C_0402_1005Metric" H 8638 3900 50  0001 C CNN
@@
 $EndComp
 $Comp
-L power:+BATT #PWR063
+L power:+BATT #PWR018
 U 1 1 5C29E17B
 P 8600 3400
-F 0 "#PWR063" H 8600 3250 50  0001 C CNN
+F 0 "#PWR018" H 8600 3250 50  0001 C CNN
 F 1 "+BATT" H 8615 3573 50  0000 C CNN
 F 2 "" H 8600 3400 50  0001 C CNN
@@
 $EndComp
 $Comp
-L power:GND #PWR064
+L power:GND #PWR019
 U 1 1 5C29E1A4
 P 8600 4600
-F 0 "#PWR064" H 8600 4350 50  0001 C CNN
+F 0 "#PWR019" H 8600 4350 50  0001 C CNN
 F 1 "GND" H 8600 4450 50  0000 C CNN
 F 2 "" H 8600 4600 50  0000 C CNN

Commit message: KiCad: update pcb
Parts:
- C4: symbol Device:C_Small -> KERISE-rescue:C_Small-Device-KERISE-rescue-KERISE-rescue
- C5: symbol Device:C -> KERISE-rescue:C-Device-KERISE-rescue-KERISE-rescue
- D1, D2, D3, D4: symbol Device:LED_Small -> KERISE-rescue:LED_Small-Device-KERISE-rescue-KERISE-rescue
- LS1: footprint mouse:SMT-0440-S-R -> mouse:SMT-0340-T-R; symbol Device:Speaker -> KERISE-rescue:Speaker-Device-KERISE-rescue-KERISE-rescue
- Q1: symbol Device:Q_NMOS_GSD -> KERISE-rescue:Q_NMOS_GSD-Device-KERISE-rescue-KERISE-rescue
- R4: symbol Device:R -> KERISE-rescue:R-Device-KERISE-rescue-KERISE-rescue
- RN1: symbol Device:R_Pack04 -> KERISE-rescue:R_Pack04-Device-KERISE-rescue-KERISE-rescue
- SW2: symbol Switch:SW_Push -> KERISE-rescue:SW_Push-Switch-KERISE-rescue-KERISE-rescue
Changed lines of the file:
@@
 $EndDescr
 $Comp
-L power:GND #PWR015
+L KERISE-rescue:GND-power-KERISE-rescue-KERISE-rescue #PWR015
 U 1 1 57CEA2EF
 P 6500 4600
@@
 User Interface
 $Comp
-L Device:Speaker LS1
+L KERISE-rescue:Speaker-Device-KERISE-rescue-KERISE-rescue LS1
 U 1 1 594AA6DF
 P 8200 3500
 F 0 "LS1" H 8250 3725 50  0000 R CNN
 F 1 "Speaker" H 8250 3650 50  0000 R CNN
-F 2 "mouse:SMT-0440-S-R" H 8200 3300 50  0001 C CNN
+F 2 "mouse:SMT-0340-T-R" H 8200 3300 50  0001 C CNN
 F 3 "" H 8190 3450 50  0001 C CNN
 	1    8200 3500
@@
 	6500 4600 6500 4400
 $Comp
-L power:GND #PWR017
+L KERISE-rescue:GND-power-KERISE-rescue-KERISE-rescue #PWR017
 U 1 1 5A1C53C4
 P 7900 4600
@@
 SDA
 $Comp
-L power:+3.3V #PWR09
+L KERISE-rescue:+3.3V-power-KERISE-rescue-KERISE-rescue #PWR?
 U 1 1 5A202D5A
 P 4050 2950
+AR Path="/5A202D5A" Ref="#PWR?"  Part="1"
+AR Path="/57CD8D81/5A202D5A" Ref="#PWR09"  Part="1"
 F 0 "#PWR09" H 4050 2800 50  0001 C CNN
 F 1 "+3.3V" H 4050 3090 50  0000 C CNN
@@
 	4050 2950 4050 3050
 $Comp
-L power:GND #PWR010
+L KERISE-rescue:GND-power-KERISE-rescue-KERISE-rescue #PWR010
 U 1 1 5A202F53
 P 4050 4650
@@
 	5050 3050 5050 2950
 $Comp
-L power:+3.3V #PWR012
+L KERISE-rescue:+3.3V-power-KERISE-rescue-KERISE-rescue #PWR?
 U 1 1 5A204571
 P 5050 2950
+AR Path="/5A204571" Ref="#PWR?"  Part="1"
+AR Path="/57CD8D81/5A204571" Ref="#PWR012"  Part="1"
 F 0 "#PWR012" H 5050 2800 50  0001 C CNN
 F 1 "+3.3V" H 5050 3090 50  0000 C CNN
@@
 $EndComp
 $Comp
-L Device:LED_Small D2
+L KERISE-rescue:LED_Small-Device-KERISE-rescue-KERISE-rescue D2
 U 1 1 5A204565
 P 5050 3150
@@
 	4750 3050 4750 2950
 $Comp
-L power:+3.3V #PWR011
+L KERISE-rescue:+3.3V-power-KERISE-rescue-KERISE-rescue #PWR?
 U 1 1 5A203D72
 P 4750 2950
+AR Path="/5A203D72" Ref="#PWR?"  Part="1"
+AR Path="/57CD8D81/5A203D72" Ref="#PWR011"  Part="1"
 F 0 "#PWR011" H 4750 2800 50  0001 C CNN
 F 1 "+3.3V" H 4750 3090 50  0000 C CNN
@@
 $EndComp
 $Comp
-L Device:LED_Small D1
+L KERISE-rescue:LED_Small-Device-KERISE-rescue-KERISE-rescue D1
 U 1 1 5A203147
 P 4750 3150
@@
 	5650 3050 5650 2950
 $Comp
-L power:+3.3V #PWR014
+L KERISE-rescue:+3.3V-power-KERISE-rescue-KERISE-rescue #PWR?
 U 1 1 5A20460C
 P 5650 2950
+AR Path="/5A20460C" Ref="#PWR?"  Part="1"
+AR Path="/57CD8D81/5A20460C" Ref="#PWR014"  Part="1"
 F 0 "#PWR014" H 5650 2800 50  0001 C CNN
 F 1 "+3.3V" H 5650 3090 50  0000 C CNN
@@
 $EndComp
 $Comp
-L Device:LED_Small D4
+L KERISE-rescue:LED_Small-Device-KERISE-rescue-KERISE-rescue D4
 U 1 1 5A204618
 P 5650 3150
@@
 	5350 3050 5350 2950
 $Comp
-L power:+3.3V #PWR013
+L KERISE-rescue:+3.3V-power-KERISE-rescue-KERISE-rescue #PWR?
 U 1 1 5A204620
 P 5350 2950
+AR Path="/5A204620" Ref="#PWR?"  Part="1"
+AR Path="/57CD8D81/5A204620" Ref="#PWR013"  Part="1"
 F 0 "#PWR013" H 5350 2800 50  0001 C CNN
 F 1 "+3.3V" H 5350 3090 50  0000 C CNN
@@
 $EndComp
 $Comp
-L Device:LED_Small D3
+L KERISE-rescue:LED_Small-Device-KERISE-rescue-KERISE-rescue D3
 U 1 1 5A20462C
 P 5350 3150
@@
 $EndComp
 $Comp
-L Device:C_Small C4
+L KERISE-rescue:C_Small-Device-KERISE-rescue-KERISE-rescue C4
 U 1 1 5A2A1F42
 P 3850 3250
@@
 $EndComp
 $Comp
-L power:GND #PWR08
+L KERISE-rescue:GND-power-KERISE-rescue-KERISE-rescue #PWR08
 U 1 1 5A2A2041
 P 3850 3350
@@
 $EndComp
 $Comp
-L Device:Q_NMOS_GSD Q1
+L KERISE-rescue:Q_NMOS_GSD-Device-KERISE-rescue-KERISE-rescue Q1
 U 1 1 5B6723D7
 P 7800 4300
@@
 	7500 4300 7600 4300
 $Comp
-L Device:R R4
+L KERISE-rescue:R-Device-KERISE-rescue-KERISE-rescue R4
 U 1 1 5B6725CD
 P 7900 3850
@@
 	7900 4000 7900 4100
 $Comp
-L Switch:SW_Push SW2
+L KERISE-rescue:SW_Push-Switch-KERISE-rescue-KERISE-rescue SW2
 U 1 1 5B6F29AF
 P 6500 4200
@@
 $EndComp
 $Comp
-L power:+BATT #PWR016
+L KERISE-rescue:+BATT-power-KERISE-rescue-KERISE-rescue #PWR016
 U 1 1 5C29DB6A
 P 7900 3400
@@
 $EndComp
 $Comp
-L Device:C C5
+L KERISE-rescue:C-Device-KERISE-rescue-KERISE-rescue C5
 U 1 1 5C29E0A6
 P 8600 4050
@@
 $EndComp
 $Comp
-L power:+BATT #PWR018
+L KERISE-rescue:+BATT-power-KERISE-rescue-KERISE-rescue #PWR018
 U 1 1 5C29E17B
 P 8600 3400
@@
 $EndComp
 $Comp
-L power:GND #PWR019
+L KERISE-rescue:GND-power-KERISE-rescue-KERISE-rescue #PWR019
 U 1 1 5C29E1A4
 P 8600 4600
@@
 	8600 3900 8600 3400
 $Comp
-L Device:R_Pack04 RN1
+L KERISE-rescue:R_Pack04-Device-KERISE-rescue-KERISE-rescue RN1
 U 1 1 5C3F6DA5
 P 5150 3650
